File: Main.kicad_sch (KiCad schematic)
At the start: 2 parts, among them J4 Conn_02x12, J5 Conn_02x12

Commit message: v2.0.0 WIP
Parts:
- renumbered J5 to J4, J4 to J5
Changed lines of the file:
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@@
 		(on_board yes)
 		(dnp no)
-		(property "Reference" "#PWR025"
+		(property "Reference" "#PWR014"
 			(at 100.33 25.4 0)
 			(effects
@@
 			(project "pico_concole_v2_daughter_board"
 				(path "/aa71e631-a14f-409f-b19b-1d980ff58830/4886cccb-afbd-4125-b9a9-e3555db25593"
-					(reference "#PWR025")
+					(reference "#PWR014")
 					(unit 1)
 				)
@@
 		(on_board yes)
 		(dnp no)
-		(property "Reference" "#PWR028"
+		(property "Reference" "#PWR016"
 			(at 118.11 64.77 0)
 			(effects
@@
 			(project "pico_concole_v2_daughter_board"
 				(path "/aa71e631-a14f-409f-b19b-1d980ff58830/4886cccb-afbd-4125-b9a9-e3555db25593"
-					(reference "#PWR028")
+					(reference "#PWR016")
 					(unit 1)
 				)
@@
 		(on_board yes)
 		(dnp no)
-		(property "Reference" "#PWR030"
+		(property "Reference" "#PWR012"
 			(at 36.83 64.77 0)
 			(effects
@@
 			(project "pico_concole_v2_daughter_board"
 				(path "/aa71e631-a14f-409f-b19b-1d980ff58830/4886cccb-afbd-4125-b9a9-e3555db25593"
-					(reference "#PWR030")
+					(reference "#PWR012")
 					(unit 1)
 				)
@@
 		(on_board yes)
 		(dnp no)
-		(property "Reference" "#PWR026"
+		(property "Reference" "#PWR017"
 			(at 120.65 29.21 0)
 			(effects
@@
 			(project "pico_concole_v2_daughter_board"
 				(path "/aa71e631-a14f-409f-b19b-1d980ff58830/4886cccb-afbd-4125-b9a9-e3555db25593"
-					(reference "#PWR026")
+					(reference "#PWR017")
 					(unit 1)
 				)
@@
 		(dnp no)
 		(fields_autoplaced yes)
-		(property "Reference" "J5"
+		(property "Reference" "J4"
 			(at 45.72 21.59 0)
 			(effects
@@
 			(project "pico_concole_v2_daughter_board"
 				(path "/aa71e631-a14f-409f-b19b-1d980ff58830/4886cccb-afbd-4125-b9a9-e3555db25593"
-					(reference "J5")
+					(reference "J4")
 					(unit 1)
 				)
@@
 		(on_board yes)
 		(dnp no)
-		(property "Reference" "#PWR027"
+		(property "Reference" "#PWR013"
 			(at 97.79 30.48 0)
 			(effects
@@
 			(project "pico_concole_v2_daughter_board"
 				(path "/aa71e631-a14f-409f-b19b-1d980ff58830/4886cccb-afbd-4125-b9a9-e3555db25593"
-					(reference "#PWR027")
+					(reference "#PWR013")
 					(unit 1)
 				)
@@
 		(dnp no)
 		(fields_autoplaced yes)
-		(property "Reference" "J4"
+		(property "Reference" "J5"
 			(at 109.22 21.59 0)
 			(effects
@@
 			(project "pico_concole_v2_daughter_board"
 				(path "/aa71e631-a14f-409f-b19b-1d980ff58830/4886cccb-afbd-4125-b9a9-e3555db25593"
-					(reference "J4")
+					(reference "J5")
 					(unit 1)
 				)
@@
 		(on_board yes)
 		(dnp no)
-		(property "Reference" "#PWR024"
+		(property "Reference" "#PWR015"
 			(at 118.11 25.4 0)
 			(effects
@@
 			(project "pico_concole_v2_daughter_board"
 				(path "/aa71e631-a14f-409f-b19b-1d980ff58830/4886cccb-afbd-4125-b9a9-e3555db25593"
-					(reference "#PWR024")
+					(reference "#PWR015")
 					(unit 1)
 				)
@@
 		(on_board yes)
 		(dnp no)
-		(property "Reference" "#PWR033"
+		(property "Reference" "#PWR011"
 			(at 36.83 29.21 0)
 			(effects
@@
 			(project "pico_concole_v2_daughter_board"
 				(path "/aa71e631-a14f-409f-b19b-1d980ff58830/4886cccb-afbd-4125-b9a9-e3555db25593"
-					(reference "#PWR033")
-					(unit 1)
-				)
+					(reference "#PWR011")
+					(unit 1)
+				)

Commit message: v2.0.0 WIP
Connections:
- net MAIN_GPIO09 renamed MAIN_GPIO9
Changed lines of the file:
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@@
 		)
 	)
-	(label "MAIN_GPIO09"
+	(label "MAIN_GPIO9"
 		(at 21.59 35.56 0)
 		(effects
@@
 		(on_board yes)
 		(dnp no)
-		(property "Reference" "#PWR014"
+		(property "Reference" "#PWR024"
 			(at 100.33 25.4 0)
 			(effects
@@
 			(project "pico_concole_v2_daughter_board"
 				(path "/aa71e631-a14f-409f-b19b-1d980ff58830/4886cccb-afbd-4125-b9a9-e3555db25593"
-					(reference "#PWR014")
+					(reference "#PWR024")
 					(unit 1)
 				)
@@
 		(on_board yes)
 		(dnp no)
-		(property "Reference" "#PWR016"
+		(property "Reference" "#PWR030"
 			(at 118.11 64.77 0)
 			(effects
@@
 			(project "pico_concole_v2_daughter_board"
 				(path "/aa71e631-a14f-409f-b19b-1d980ff58830/4886cccb-afbd-4125-b9a9-e3555db25593"
-					(reference "#PWR016")
+					(reference "#PWR030")
 					(unit 1)
 				)
@@
 		(on_board yes)
 		(dnp no)
-		(property "Reference" "#PWR012"
+		(property "Reference" "#PWR029"
 			(at 36.83 64.77 0)
 			(effects
@@
 			(project "pico_concole_v2_daughter_board"
 				(path "/aa71e631-a14f-409f-b19b-1d980ff58830/4886cccb-afbd-4125-b9a9-e3555db25593"
-					(reference "#PWR012")
+					(reference "#PWR029")
 					(unit 1)
 				)
@@
 		(on_board yes)
 		(dnp no)
-		(property "Reference" "#PWR017"
+		(property "Reference" "#PWR027"
 			(at 120.65 29.21 0)
 			(effects
@@
 			(project "pico_concole_v2_daughter_board"
 				(path "/aa71e631-a14f-409f-b19b-1d980ff58830/4886cccb-afbd-4125-b9a9-e3555db25593"
-					(reference "#PWR017")
+					(reference "#PWR027")
 					(unit 1)
 				)
@@
 		(on_board yes)
 		(dnp no)
-		(property "Reference" "#PWR013"
+		(property "Reference" "#PWR028"
 			(at 97.79 30.48 0)
 			(effects
@@
 			(project "pico_concole_v2_daughter_board"
 				(path "/aa71e631-a14f-409f-b19b-1d980ff58830/4886cccb-afbd-4125-b9a9-e3555db25593"
-					(reference "#PWR013")
+					(reference "#PWR028")
 					(unit 1)
 				)
@@
 		(on_board yes)
 		(dnp no)
-		(property "Reference" "#PWR015"
+		(property "Reference" "#PWR025"
 			(at 118.11 25.4 0)
 			(effects
@@
 			(project "pico_concole_v2_daughter_board"
 				(path "/aa71e631-a14f-409f-b19b-1d980ff58830/4886cccb-afbd-4125-b9a9-e3555db25593"
-					(reference "#PWR015")
+					(reference "#PWR025")
 					(unit 1)
 				)
@@
 		(on_board yes)
 		(dnp no)
-		(property "Reference" "#PWR011"
+		(property "Reference" "#PWR026"
 			(at 36.83 29.21 0)
 			(effects
@@
 			(project "pico_concole_v2_daughter_board"
 				(path "/aa71e631-a14f-409f-b19b-1d980ff58830/4886cccb-afbd-4125-b9a9-e3555db25593"
-					(reference "#PWR011")
+					(reference "#PWR026")
 					(unit 1)
 				)
