File: Daughterboard.kicad_sch (KiCad schematic)
At the start: 87 parts, among them SW1 SW_Push, SW10 SW_Push, SW11 SW_Push, SW12 SW_Push, SW13 SW_Push, SW14 SW_Push, SW15 SW_Push, SW16 SW_Push, SW17 SW_Push, SW2 SW_Push, SW3 SW_Push, SW4 SW_Push, SW5 SW_Push, SW6 SW_Push, SW7 SW_Push, SW8 SW_Push, SW9 SW_Push, U1 PCM5102A, U2 PAM8403D, U4 TSOP34S40F, U5 XPT2046TS

Commit message: Place components temporarily
Parts:
- removed H15, H16: M2, MountingHole:MountingHole_2.2mm_M2, symbol Mechanical:MountingHole
- SW1, SW3: footprint (none) -> Button_Switch_THT:SM-05H-0xC-Zippy
- SW10, SW11, SW12, SW13, SW14, SW15, SW16, SW5, SW6, SW7, SW8, SW9: footprint (none) -> Button_Switch_THT:SW_PUSH_6mm_H7.3mm
- SW17: footprint (none) -> Button_Switch_SMD:SW_SPST_PTS810
- SW2, SW4: footprint (none) -> Button_Switch_THT:SM-05H-0xD-Zippy
Other:
- moved on the sheet: BAT1

Commit message: Place components temporarily
Parts:
- D1, D10, D11, D12, D13, D14, D15, D16, D2, D3, D4, D5, D6, D7, D8, D9: footprint (none) -> Diode_SMD:D_0805_2012Metric_Pad1.15x1.40mm_HandSolder
- JOY1, JOY2: footprint (none) -> Connector_FFC-FPC:TE_0-1734839-5_1x05-1MP_P0.5mm_Horizontal
Changed lines of the file:
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@@
 			)
 		)
-		(property "Footprint" ""
+		(property "Footprint" "Diode_SMD:D_0805_2012Metric_Pad1.15x1.40mm_HandSolder"
 			(at 181.61 273.05 90)
 			(effects
@@
 			)
 		)
-		(property "Footprint" ""
+		(property "Footprint" "Diode_SMD:D_0805_2012Metric_Pad1.15x1.40mm_HandSolder"
 			(at 166.37 242.57 90)
 			(effects
@@
 			)
 		)
-		(property "Footprint" ""
+		(property "Footprint" "Diode_SMD:D_0805_2012Metric_Pad1.15x1.40mm_HandSolder"
 			(at 151.13 257.81 90)
 			(effects
@@
 			)
 		)
-		(property "Footprint" ""
+		(property "Footprint" "Diode_SMD:D_0805_2012Metric_Pad1.15x1.40mm_HandSolder"
 			(at 181.61 242.57 90)
 			(effects
@@
 			)
 		)
-		(property "Footprint" ""
+		(property "Footprint" "Diode_SMD:D_0805_2012Metric_Pad1.15x1.40mm_HandSolder"
 			(at 151.13 227.33 90)
 			(effects
@@
 			)
 		)
-		(property "Footprint" ""
+		(property "Footprint" "Connector_FFC-FPC:TE_0-1734839-5_1x05-1MP_P0.5mm_Horizontal"
 			(at 109.22 257.81 0)
 			(effects
@@
 			)
 		)
-		(property "Footprint" ""
+		(property "Footprint" "Diode_SMD:D_0805_2012Metric_Pad1.15x1.40mm_HandSolder"
 			(at 151.13 242.57 90)
 			(effects
@@
 			)
 		)
-		(property "Footprint" ""
+		(property "Footprint" "Diode_SMD:D_0805_2012Metric_Pad1.15x1.40mm_HandSolder"
 			(at 135.89 257.81 90)
 			(effects
@@
 			)
 		)
-		(property "Footprint" ""
+		(property "Footprint" "Diode_SMD:D_0805_2012Metric_Pad1.15x1.40mm_HandSolder"
 			(at 135.89 242.57 90)
 			(effects
@@
 			)
 		)
-		(property "Footprint" ""
+		(property "Footprint" "Diode_SMD:D_0805_2012Metric_Pad1.15x1.40mm_HandSolder"
 			(at 166.37 257.81 90)
 			(effects
@@
 			)
 		)
-		(property "Footprint" ""
+		(property "Footprint" "Diode_SMD:D_0805_2012Metric_Pad1.15x1.40mm_HandSolder"
 			(at 181.61 257.81 90)
 			(effects
@@
 			)
 		)
-		(property "Footprint" ""
+		(property "Footprint" "Diode_SMD:D_0805_2012Metric_Pad1.15x1.40mm_HandSolder"
 			(at 151.13 273.05 90)
 			(effects
@@
 			)
 		)
-		(property "Footprint" ""
+		(property "Footprint" "Diode_SMD:D_0805_2012Metric_Pad1.15x1.40mm_HandSolder"
 			(at 166.37 227.33 90)
 			(effects
@@
 			)
 		)
-		(property "Footprint" ""
+		(property "Footprint" "Connector_FFC-FPC:TE_0-1734839-5_1x05-1MP_P0.5mm_Horizontal"
 			(at 109.22 227.33 0)
 			(effects
@@
 			)
 		)
-		(property "Footprint" ""
+		(property "Footprint" "Diode_SMD:D_0805_2012Metric_Pad1.15x1.40mm_HandSolder"
 			(at 135.89 273.05 90)
 			(effects
@@
 			)
 		)
-		(property "Footprint" ""
+		(property "Footprint" "Diode_SMD:D_0805_2012Metric_Pad1.15x1.40mm_HandSolder"
 			(at 166.37 273.05 90)
 			(effects
@@
 			)
 		)
-		(property "Footprint" ""
+		(property "Footprint" "Diode_SMD:D_0805_2012Metric_Pad1.15x1.40mm_HandSolder"
 			(at 135.89 227.33 90)
 			(effects
@@
 			)
 		)
-		(property "Footprint" ""
+		(property "Footprint" "Diode_SMD:D_0805_2012Metric_Pad1.15x1.40mm_HandSolder"
 			(at 181.61 227.33 90)
 			(effects

Commit message: v2.0.0 WIP
Parts:
- removed H13, H14: M2, MountingHole:MountingHole_2.2mm_M2, symbol Mechanical:MountingHole
- added C1, C6, C7: 1u, Capacitor_SMD:C_0402_1005Metric_Pad0.74x0.62mm_HandSolder, symbol Device:C
- added C2, C3: 470n, Capacitor_SMD:C_0402_1005Metric_Pad0.74x0.62mm_HandSolder, symbol Device:C
- added C4, C5: 470u, Capacitor_SMD:C_0402_1005Metric_Pad0.74x0.62mm_HandSolder, symbol Device:C
- added R10, R9: 1k, Resistor_SMD:R_0603_1608Metric_Pad0.98x0.95mm_HandSolder, symbol Device:R
Connections:
- net I2S_DATA is gone; now on net GPIO36: U1.14 (DIN)
- net I2S_LRCK is gone; now on net GPIO38: U1.15 (LRCK)
- net I2S_SCK is gone; now on net GPIO37: U1.13 (BCK)
- net Joy1_BTN is gone; now on net GPIO26: JOY1.3 (Pin_3)
- net Joy1_X is gone; now on net GPIO40_ADC0: JOY1.5 (Pin_5)
- net Joy1_Y is gone; now on net GPIO41_ADC1: JOY1.2 (Pin_2)
- net Joy2_BTN is gone; now on net GPIO27: JOY2.3 (Pin_3)
- net Joy2_X is gone; now on net GPIO42_ADC2: JOY2.5 (Pin_5)
- net Joy2_Y is gone; now on net GPIO43_ADC3: JOY2.2 (Pin_2)
- net TOUCH_MISO is gone; now on net MAIN_GPIO20: U5.12 (DOUT)
- net TOUCH_MOSI is gone; now on net MAIN_GPIO23: U5.14 (DIN)
- net TOUCH_SCK is gone; now on net MAIN_GPIO22: U5.16 (DCLK)
- net ~{AMP_MUTE} is gone; now on net GPIO39: U1.17 (XSMT)
- net ~{TOUCH_CS} is gone; now on net MAIN_GPIO21: U5.15 (~{CS})
- net ~{TOUCH_IRQ} is gone; now on net MAIN_GPIO24: U5.11 (~{PENIRQ})
- net +3V3: now also DP1.12 (Pin_12), DP1.6 (Pin_6), DP1.7 (Pin_7)
- net DP_DC: now also DP1.10 (Pin_10)
- net DP_MISO: now also DP1.14 (Pin_14)
- net DP_MOSI: now also DP1.13 (Pin_13)
- net DP_SCK: now also DP1.11 (Pin_11)
- net GNDA: now also U2.11 (GND), U2.15 (PGND), U2.2 (PGND), C1.2, C4.2, C5.2, C6.2, C7.2
- net MAIN_GPIO14: now also DP1.9 (Pin_9)
- net MAIN_GPIO15: now also DP1.15 (Pin_15)
- net SPK_L: now also C2.1; no longer U2.7 (INL)
- net SPK_R: now also C3.1; no longer U2.10 (INR)
- net TP_X+: now also DP1.3 (Pin_3)
- net TP_X-: now also DP1.1 (Pin_1)
- net TP_Y+: now also DP1.2 (Pin_2)
- net TP_Y-: now also DP1.4 (Pin_4)
- net VIN: now also U2.13 (PVDD), U2.4 (PVDD), U2.6 (VDD), C4.1, C5.1, C6.1, C7.1, R10.1, R9.1
- net at U2.12 (~{SHDN}): now also R10.2
- net at U2.5 (~{MUTE}): now also R9.2
- net at U2.8 (VREF): now also C1.1
- new net: C2.2, U2.7 (INL)
- new net: C3.2, U2.10 (INR)
- no-connect marks 0 -> 2
Other:
- moved on the sheet: AUDIO1, DP1, LED5, LRA1, LRA2, R4, SPK1, SPK2, U1, U2, U4, U5

Commit message: v2.0.0 WIP
Parts:
- added C10, C13, C14: 1u, Capacitor_SMD:C_0402_1005Metric_Pad0.74x0.62mm_HandSolder, symbol Device:C
- added C11, C12: 470u, Capacitor_SMD:C_0402_1005Metric_Pad0.74x0.62mm_HandSolder, symbol Device:C
- added C8, C9: 470n, Capacitor_SMD:C_0402_1005Metric_Pad0.74x0.62mm_HandSolder, symbol Device:C
- added R11, R12: 1k, Resistor_SMD:R_0603_1608Metric_Pad0.98x0.95mm_HandSolder, symbol Device:R
- added TP11, TP12, TP13, TP14, TP15, TP16, TP17, TP18, TP19, TP20, TP21, TP22, TP23: TP, TestPoint:TestPoint_Pad_1.0x1.0mm, symbol Connector:TestPoint
- added U6: PAM8403D, Package_SO:SOIC-16_3.9x9.9mm_P1.27mm, symbol Amplifier_Audio:PAM8403D
- renumbered C2 to C1, C3 to C2, C1 to C3, D7 to D10, D15 to D12, D4 to D13, D8 to D14, D12 to D15, D5 to D2, D9 to D3, D13 to D4, D2 to D5, D10 to D7, D14 to D8, D3 to D9, H4 to H10, H8 to H11, H5 to H2, H9 to H3, H2 to H4, H6 to H5, H10 to H6, H3 to H7, H7 to H8, H11 to H9, R5 to R3, R6 to R4, R7 to R5, R8 to R6, R3 to R7, R4 to R8, SW17 to SW1, SW3 to SW10, SW7 to SW11, SW11 to SW12, SW15 to SW13, SW4 to SW14, SW8 to SW15, SW12 to SW16, SW16 to SW17, SW1 to SW2, SW5 to SW3, SW9 to SW4, SW13 to SW5, SW2 to SW6, SW6 to SW7, SW10 to SW8, SW14 to SW9, TP9 to TP1, TP1 to TP2, TP5 to TP4, TP7 to TP5, TP2 to TP6, TP4 to TP7, TP6 to TP8, TP8 to TP9, U1 to U2, U4 to U3, U5 to U4, U2 to U5
Connections:
- net +3V3: now also DP1.1 (Pin_1), DP1.2 (Pin_2), DP1.29 (Pin_29), DP1.3 (Pin_3), DP1.34 (Pin_34), DP1.35 (Pin_35); no longer DP1.12 (Pin_12), DP1.38 (Pin_38), DP1.39 (Pin_39), DP1.40 (Pin_40), DP1.6 (Pin_6), DP1.7 (Pin_7)
- net DP_DC: now also DP1.31 (Pin_31); no longer DP1.10 (Pin_10)
- net DP_MISO: now also DP1.27 (Pin_27); no longer DP1.14 (Pin_14)
- net DP_MOSI: now also DP1.28 (Pin_28); no longer DP1.13 (Pin_13)
- net DP_SCK: now also DP1.30 (Pin_30); no longer DP1.11 (Pin_11)
- net GND: now also DP1.10 (Pin_10), DP1.11 (Pin_11), DP1.12 (Pin_12), DP1.13 (Pin_13), DP1.14 (Pin_14), DP1.15 (Pin_15), DP1.36 (Pin_36), DP1.4 (Pin_4), DP1.9 (Pin_9); no longer DP1.26 (Pin_26), DP1.27 (Pin_27), DP1.28 (Pin_28), DP1.29 (Pin_29), DP1.30 (Pin_30), DP1.31 (Pin_31), DP1.32 (Pin_32), DP1.37 (Pin_37), DP1.5 (Pin_5)
- net GNDA: now also C10.2, C11.2, C12.2, C13.2, C14.2, U6.11 (GND), U6.15 (PGND), U6.2 (PGND)
- net GPIO10: now also C2.1
- net GPIO12: now also TP11.1
- net GPIO13: now also TP12.1
- net GPIO14: now also TP13.1
- net GPIO15: now also TP14.1
- net GPIO16: now also TP15.1
- net GPIO17: now also TP16.1
- net GPIO18: now also TP17.1
- net GPIO19: now also TP18.1
- net GPIO6: now also TP19.1
- net GPIO7: now also TP20.1
- net GPIO8: now also C8.1
- net LRA_L+: now also U6.1 (LOUT+)
- net LRA_L-: now also U6.3 (LOUT-)
- net LRA_R+: now also U5.16 (ROUT+)
- net LRA_R-: now also U5.14 (ROUT-)
- net MAIN_GPIO10: now also TP21.1
- net MAIN_GPIO11: now also TP22.1
- net MAIN_GPIO14: now also DP1.32 (Pin_32); no longer DP1.9 (Pin_9)
- net MAIN_GPIO15: now also DP1.26 (Pin_26); no longer DP1.15 (Pin_15)
- net SPK_L: now also C9.1; no longer C1.1
- net SPK_L+: now also U6.16 (ROUT+); no longer U5.1 (LOUT+)
- net SPK_L-: now also U6.14 (ROUT-); no longer U5.3 (LOUT-)
- net SPK_R: now also C1.1; no longer C2.1
- net SPK_R+: now also U5.1 (LOUT+); no longer U5.16 (ROUT+)
- net SPK_R-: now also U5.3 (LOUT-); no longer U5.14 (ROUT-)
- net TP_X+: now also DP1.38 (Pin_38); no longer DP1.3 (Pin_3)
- net TP_X-: now also DP1.40 (Pin_40); no longer DP1.1 (Pin_1)
- net TP_Y+: now also DP1.39 (Pin_39); no longer DP1.2 (Pin_2)
- net TP_Y-: now also DP1.37 (Pin_37); no longer DP1.4 (Pin_4)
- net VIN: now also C11.1, C12.1, C13.1, C14.1, R11.1, R12.1, U6.13 (PVDD), U6.4 (PVDD), U6.6 (VDD)
- net GPIO40_ADC0 renamed GPIO40
- net GPIO41_ADC1 renamed GPIO41
- net GPIO42_ADC2 renamed GPIO42
- net GPIO43_ADC3 renamed GPIO43
- new net: C10.1, U6.8 (VREF)
- new net: R12.2, U6.12 (~{SHDN})
- new net: DP1.5 (Pin_5), DP1.6 (Pin_6), DP1.7 (Pin_7)
- new net: C8.2, U6.7 (INL)
- new net: C9.2, U6.10 (INR)
- new net: R11.2, U6.5 (~{MUTE})
- new net GPIO47: TP23.1
Other:
- note added: "1"
- note added: "40"
- note added: "AMP (L)"
- note added: "AMP (R)"
- note added: "Connectors"
- note removed: "Vibration (LRA)"
- moved on the sheet: AUDIO1, C1, C2, C3, C4, C5, C6, C7, DP1, H1, H10, H11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

Commit message: v2.0.0 WIP
Parts:
- added C19, C20: 1u, Capacitor_SMD:C_0402_1005Metric_Pad0.74x0.62mm_HandSolder, symbol Device:C
- added R11, R18, R19: 1k, Resistor_SMD:R_0402_1005Metric_Pad0.72x0.64mm_HandSolder, symbol Device:R
- added R16, R17: 330k, Resistor_SMD:R_0402_1005Metric_Pad0.72x0.64mm_HandSolder, symbol Device:R
- added TP1, TP25, TP26, TP27, TP28, TP29, TP30: TP, TestPoint:TestPoint_Pad_1.0x1.0mm, symbol Connector:TestPoint
- R10: renamed from R7; footprint Resistor_SMD:R_0805_2012Metric_Pad1.20x1.40mm_HandSolder -> Resistor_SMD:R_0402_1005Metric_Pad0.72x0.64mm_HandSolder
- R12: renamed from R9; footprint Resistor_SMD:R_0603_1608Metric_Pad0.98x0.95mm_HandSolder -> Resistor_SMD:R_0402_1005Metric_Pad0.72x0.64mm_HandSolder
- R13: renamed from R10; footprint Resistor_SMD:R_0603_1608Metric_Pad0.98x0.95mm_HandSolder -> Resistor_SMD:R_0402_1005Metric_Pad0.72x0.64mm_HandSolder
- R14: renamed from R11; footprint Resistor_SMD:R_0603_1608Metric_Pad0.98x0.95mm_HandSolder -> Resistor_SMD:R_0402_1005Metric_Pad0.72x0.64mm_HandSolder
- R15: renamed from R12; footprint Resistor_SMD:R_0603_1608Metric_Pad0.98x0.95mm_HandSolder -> Resistor_SMD:R_0402_1005Metric_Pad0.72x0.64mm_HandSolder
- R9: renamed from R8; footprint Resistor_SMD:R_0805_2012Metric_Pad1.20x1.40mm_HandSolder -> Resistor_SMD:R_0402_1005Metric_Pad0.72x0.64mm_HandSolder
- renumbered C1 to C21, C8 to C22, C2 to C23, C9 to C24, C3 to C25, C10 to C26, C4 to C27, C5 to C28, C6 to C29, C7 to C30, C11 to C31, C12 to C32, C13 to C33, C14 to C34, D7 to D10, D15 to D12, D4 to D13, D8 to D14, D12 to D15, D5 to D2, D9 to D3, D13 to D4, D2 to D5, D10 to D7, D14 to D8, D3 to D9, H11 to H10, H6 to H11, H7 to H2, H2 to H3, H8 to H4, H3 to H5, H9 to H6, H4 to H7, H10 to H8, H5 to H9, LED5 to LED1, LED1 to LED2, LED2 to LED3, LED3 to LED4, LED4 to LED5, R3 to R20, R4 to R21, R5 to R22, R6 to R23, SW11 to SW10, SW15 to SW11, SW4 to SW12, SW8 to SW13, SW12 to SW14, SW16 to SW15, SW5 to SW16, SW9 to SW17, SW13 to SW18, SW17 to SW19, SW1 to SW3, SW2 to SW4, SW6 to SW5, SW10 to SW6, SW14 to SW7, SW3 to SW8, SW7 to SW9, TP15 to TP10, TP16 to TP11, TP17 to TP12, TP18 to TP13, TP23 to TP14, TP2 to TP15, TP6 to TP16, TP3 to TP17, TP7 to TP18, TP4 to TP19, TP21 to TP2, TP8 to TP20, TP5 to TP21, TP9 to TP22, TP1 to TP23, TP10 to TP24, TP22 to TP3, TP19 to TP4, TP20 to TP5, TP11 to TP6, TP12 to TP7, TP13 to TP8, TP14 to TP9, U2 to U5, U5 to U6, U6 to U7
Connections:
- net +3V3: now also C19.1, C20.1
- net DP_DC: now also TP29.1
- net DP_MISO: now also TP26.1
- net DP_MOSI: now also TP27.1
- net DP_SCK: now also TP28.1
- net GND: now also C19.2, C20.2
- net GPIO10: now also R18.1; no longer C23.1
- net GPIO8: now also R17.1; no longer C22.1
- net MAIN_GPIO14: now also TP30.1
- net MAIN_GPIO15: now also TP25.1
- net MAIN_GPIO25: now also R11.1
- net SPK_L: now also R19.1; no longer C24.1
- net SPK_R: now also R16.1; no longer C21.1
- new net: C22.1, R17.2
- new net: C21.1, R16.2
- new net: C23.1, R18.2
- new net: C24.1, R19.2
- new net MAIN_GPIO9: TP1.1
- new net ~{SB_RUN}: R11.2
- no-connect marks 2 -> 1
Other:
- moved on the sheet: AUDIO1, BAT1, C21, C22, C23, C24, C25, C26, C27, C28, C29, C30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

Commit message: v2.0.0 WIP
Changed lines of the file:
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@@
 	(text "AMP (R)"
 		(exclude_from_sim no)
-		(at 363.22 158.75 0)
+		(at 273.812 159.004 0)
 		(effects
 			(font
@@
 	(text "AMP (L)"
 		(exclude_from_sim no)
-		(at 275.336 159.258 0)
+		(at 362.204 159.258 0)
 		(effects
 			(font

Commit message: V2.0.0 WIP
Parts:
- removed TP10, TP12, TP13, TP6, TP7, TP8: TP, TestPoint:TestPoint_Pad_1.0x1.0mm, symbol Connector:TestPoint
- added J6: Conn_01x10_MountingPin, Connector_FFC-FPC:TE_1-1734839-0_1x10-1MP_P0.5mm_Horizontal, symbol Connector_Generic_MountingPin:Conn_01x10_MountingPin
- added TP14, TP16, TP17, TP18, TP25, TP26, TP27: TP, TestPoint:TestPoint_Pad_D1.0mm, symbol Connector:TestPoint
- SW3: footprint Button_Switch_SMD:SW_SPST_PTS810 -> Button_Switch_SMD:SW_Push_1P1T_NO_Vertical_Wuerth_434133025816
- TP1, TP11, TP2, TP3, TP4, TP9: footprint TestPoint:TestPoint_Pad_1.0x1.0mm -> TestPoint:TestPoint_Pad_D1.0mm
- TP10: renamed from TP27; footprint TestPoint:TestPoint_Pad_1.0x1.0mm -> TestPoint:TestPoint_Pad_D1.0mm
- TP12: renamed from TP26; footprint TestPoint:TestPoint_Pad_1.0x1.0mm -> TestPoint:TestPoint_Pad_D1.0mm
- TP13: renamed from TP25; footprint TestPoint:TestPoint_Pad_1.0x1.0mm -> TestPoint:TestPoint_Pad_D1.0mm
- TP15: renamed from TP14; footprint TestPoint:TestPoint_Pad_1.0x1.0mm -> TestPoint:TestPoint_Pad_D1.0mm
- TP19: renamed from TP15; footprint TestPoint:TestPoint_Pad_1.5x1.5mm -> TestPoint:TestPoint_Pad_1.0x1.0mm
- TP20: renamed from TP16; footprint TestPoint:TestPoint_Pad_1.5x1.5mm -> TestPoint:TestPoint_Pad_1.0x1.0mm
- TP21: renamed from TP17; footprint TestPoint:TestPoint_Pad_1.5x1.5mm -> TestPoint:TestPoint_Pad_1.0x1.0mm
- TP22: renamed from TP18; footprint TestPoint:TestPoint_Pad_1.5x1.5mm -> TestPoint:TestPoint_Pad_1.0x1.0mm
- TP23: renamed from TP19; footprint TestPoint:TestPoint_Pad_1.5x1.5mm -> TestPoint:TestPoint_Pad_1.0x1.0mm
- TP24: renamed from TP20; footprint TestPoint:TestPoint_Pad_1.5x1.5mm -> TestPoint:TestPoint_Pad_1.0x1.0mm
- TP28: renamed from TP21; footprint TestPoint:TestPoint_Pad_1.5x1.5mm -> TestPoint:TestPoint_Pad_1.0x1.0mm
- TP29: renamed from TP22; footprint TestPoint:TestPoint_Pad_1.5x1.5mm -> TestPoint:TestPoint_Pad_1.0x1.0mm
- TP30: renamed from TP23; footprint TestPoint:TestPoint_Pad_1.5x1.5mm -> TestPoint:TestPoint_Pad_1.0x1.0mm
- TP31: renamed from TP24; footprint TestPoint:TestPoint_Pad_1.5x1.5mm -> TestPoint:TestPoint_Pad_1.0x1.0mm
- TP5: renamed from TP30; footprint TestPoint:TestPoint_Pad_1.0x1.0mm -> TestPoint:TestPoint_Pad_D1.0mm
- TP6: renamed from TP5; footprint TestPoint:TestPoint_Pad_1.0x1.0mm -> TestPoint:TestPoint_Pad_D1.0mm
- TP7: renamed from TP29; footprint TestPoint:TestPoint_Pad_1.0x1.0mm -> TestPoint:TestPoint_Pad_D1.0mm
- TP8: renamed from TP28; footprint TestPoint:TestPoint_Pad_1.0x1.0mm -> TestPoint:TestPoint_Pad_D1.0mm
- renumbered C22 to C21, C21 to C22, C24 to C23, C23 to C24, C26 to C25, C25 to C26, C31 to C27, C32 to C28, C33 to C29, C34 to C30, C27 to C31, C28 to C32, C29 to C33, C30 to C34, R14 to R12, R15 to R13, R12 to R14, R13 to R15, R17 to R16, R16 to R17, R19 to R18, R18 to R19, U3 to U4, U4 to U5, U5 to U6, U6 to U8
Connections:
- net GNDA is gone; now on net GND: AUDIO1.S, C25.2, C26.2, C27.2, C28.2, C29.2, C30.2, C31.2, C32.2, C33.2, C34.2, U7.11 (GND), U7.15 (PGND), U7.2 (PGND), U8.11 (GND), U8.15 (PGND), U8.2 (PGND)
- net VIN is gone; now on net +3V3: C27.1, C28.1, C29.1, C30.1, C31.1, C32.1, C33.1, C34.1, R12.1, R13.1, R14.1, R15.1, TP30.1, U7.13 (PVDD), U7.4 (PVDD), U7.6 (VDD), U8.13 (PVDD), U8.4 (PVDD), U8.6 (VDD)
- net +3V3: now also U6.1 (CPVDD), U6.8 (AVDD), J6.9 (Pin_9)
- net DP_BL: now also TP14.1
- net GND: now also U6.19 (DGND), U6.3 (CPGND), U6.9 (AGND), J6.10 (Pin_10), J6.MP (MountPin)
- net GPIO10: now also TP9.1; no longer R19.1
- net GPIO11: now also TP11.1
- net GPIO12: now also J6.1 (Pin_1)
- net GPIO13: now also J6.2 (Pin_2)
- net GPIO14: now also J6.3 (Pin_3)
- net GPIO15: now also J6.4 (Pin_4); no longer TP9.1
- net GPIO16: now also J6.5 (Pin_5)
- net GPIO17: now also J6.6 (Pin_6); no longer TP11.1
- net GPIO18: now also J6.7 (Pin_7)
- net GPIO19: now also J6.8 (Pin_8)
- net GPIO26: now also TP17.1
- net GPIO27: now also TP26.1
- net GPIO40: now also TP18.1
- net GPIO41: now also TP16.1
- net GPIO42: now also TP27.1
- net GPIO43: now also TP25.1
- net GPIO9: now also R19.1
- net DP_LED_K: now reaches DP1.5 (Pin_5), DP1.6 (Pin_6), DP1.7 (Pin_7)
- net DP_LED_A: now reaches DP1.8 (Pin_8)
- no-connect marks 1 -> 2
Other:
- moved on the sheet: C19, C20, C21, C22, C23, C24, C25, C26, C27, C28, C29, C30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
