File: Daughterboard.kicad_sch (KiCad schematic)
At the start: 131 parts, among them J6 Conn_01x10_MountingPin, SW10 SW_Push, SW11 SW_Push, SW12 SW_Push, SW13 SW_Push, SW14 SW_Push, SW15 SW_Push, SW16 SW_Push, SW17 SW_Push, SW18 SW_Push, SW19 SW_Push, SW3 SW_Push, SW4 SW_Push, SW5 SW_Push, SW6 SW_Push, SW7 SW_Push, SW8 SW_Push, SW9 SW_Push, U4 TSOP34S40F, U5 XPT2046TS, U6 PCM5102A, U7 PAM8403D, U8 PAM8403D

Commit message: V2.0.0 WIP
Parts:
- added C35, C36, C41: 1u, Capacitor_SMD:C_0402_1005Metric_Pad0.74x0.62mm_HandSolder, symbol Device:C
- added C37, C38, C39, C40: 2.2u, Capacitor_SMD:C_0402_1005Metric_Pad0.74x0.62mm_HandSolder, symbol Device:C
- added JP5, JP6: Jumper_2_Small_Bridged, symbol Jumper:Jumper_2_Small_Bridged
- added R24, R25: 470, Resistor_SMD:R_0402_1005Metric_Pad0.72x0.64mm_HandSolder, symbol Device:R
- added R26: 0, Resistor_SMD:R_0402_1005Metric_Pad0.72x0.64mm_HandSolder, symbol Device:R
- R18, R19: value 1k -> 100k
Connections:
- net +3V3: now also C35.1, C36.1, C41.1, JP5.1 (A); no longer U6.8 (AVDD), U7.13 (PVDD), U7.4 (PVDD), U8.13 (PVDD), U8.4 (PVDD)
- net BTN_V1: now also SW5.1; no longer SW4.1
- net BTN_V2: now also SW4.1, SW6.1; no longer SW17.1, SW5.1
- net BTN_V3: now also SW17.1; no longer SW6.1
- net GND: now also C35.2, C36.2, C41.2, JP6.1 (A); no longer AUDIO1.S, U6.9 (AGND), U7.15 (PGND), U7.2 (PGND), U8.15 (PGND), U8.2 (PGND)
- net MAIN_GPIO25: now also R11.2; no longer R11.1
- net ~{SB_RUN}: now also R11.1; no longer R11.2
- net at SW7.2: now also D16.2 (A); no longer D4.2 (A)
- net at SW9.2: now also D2.2 (A); no longer D6.2 (A)
- net at SW19.2: now also D8.2 (A); no longer D16.2 (A)
- net at D7.2 (A): now also SW17.2; no longer SW10.2
- net at SW4.2: now also D6.2 (A); no longer D1.2 (A)
- net at D14.2 (A): now also SW6.2; no longer SW17.2
- net at SW11.2: now also D4.2 (A); no longer D8.2 (A)
- net at SW5.2: now also D5.2 (A); no longer D2.2 (A)
- net at SW8.2: now also D1.2 (A); no longer D5.2 (A)
- net at D3.2 (A): now also SW10.2; no longer SW6.2
- net at U6.2 (CAPP): now also C37.1
- net at U6.4 (CAPM): now also C37.2
- net AMP_L: no longer names the net of U6.6 (OUTL)
- net AMP_L: now also R24.1; no longer AUDIO1.R
- net AMP_R: no longer names the net of U6.7 (OUTR)
- net AMP_R: now also R25.1; no longer AUDIO1.T
- new net AGND: AUDIO1.S, C39.2, C40.2, JP6.2 (B), U6.9 (AGND), U7.15 (PGND), U7.2 (PGND), U8.15 (PGND), U8.2 (PGND)
- new net AVDD: JP5.2 (B), U6.8 (AVDD), U7.13 (PVDD), U7.4 (PVDD), U8.13 (PVDD), U8.4 (PVDD)
- new net DAC_L: AUDIO1.R, C39.1, R24.2
- new net DAC_R: AUDIO1.T, C40.1, R25.2
Other:
- moved on the sheet: LED1, R11, R9, SW10, SW11, SW17, SW19, SW4, SW5, SW6, SW7, SW8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

Commit message: v2.0.0 WIP
Parts:
- removed JP5: Jumper_2_Small_Bridged, symbol Jumper:Jumper_2_Small_Bridged
- removed R26: 0, Resistor_SMD:R_0402_1005Metric_Pad0.72x0.64mm_HandSolder, symbol Device:R
- added C42: 1u, Capacitor_SMD:C_0402_1005Metric_Pad0.74x0.62mm_HandSolder, symbol Device:C
- added C43, C45: 10u, Capacitor_SMD:C_0402_1005Metric_Pad0.74x0.62mm_HandSolder, symbol Device:C
- added C44: 47n, Capacitor_SMD:C_0402_1005Metric_Pad0.74x0.62mm_HandSolder, symbol Device:C
- added C46: 4.7u, Capacitor_SMD:C_0402_1005Metric_Pad0.74x0.62mm_HandSolder, symbol Device:C
- added FB1, FB2, FB3: FerriteBead_Small, symbol Device:FerriteBead_Small
- added J7: Conn_01x04_MountingPin, Connector_JST:JST_SH_SM04B-SRSS-TB_1x04-1MP_P1.00mm_Horizontal, symbol Connector_Generic_MountingPin:Conn_01x04_MountingPin
- added JP7, JP8: Jumper_2_Small_Bridged, symbol Jumper:Jumper_2_Small_Bridged
- added L2: 1u, symbol Device:L
- added LED6: GREEN, LED_SMD:LED_0805_2012Metric_Pad1.15x1.40mm_HandSolder, symbol Device:LED
- added R27, R28, R29, R30, R31, R32, R33: 10k, Resistor_SMD:R_0402_1005Metric_Pad0.72x0.64mm_HandSolder, symbol Device:R
- added R34: 1k, Resistor_SMD:R_0402_1005Metric_Pad0.72x0.64mm_HandSolder, symbol Device:R
- added TEMP1: temperture, Connector_Molex:Molex_PicoBlade_53261-0271_1x02-1MP_P1.25mm_Horizontal, symbol Connector_Generic_MountingPin:Conn_01x02_MountingPin
- added TP32, TP33, TP34: TP, TestPoint:TestPoint_Pad_D1.0mm, symbol Connector:TestPoint
- added U10: BQ25619, Package_DFN_QFN:Texas_RTW_WQFN-24-1EP_4x4mm_P0.5mm_EP2.7x2.7mm, symbol New_Library:BQ25619
- added U9: MPU-6050, Sensor_Motion:InvenSense_QFN-24_4x4mm_P0.5mm, symbol Sensor_Motion:MPU-6050
- R12, R13, R14, R15: value 1k -> 10k
- R20, R21, R22, R23: footprint Resistor_SMD:R_0805_2012Metric_Pad1.20x1.40mm_HandSolder -> Resistor_SMD:R_0402_1005Metric_Pad0.72x0.64mm_HandSolder
Connections:
- net +3V3: now also FB1.1, FB2.1, FB3.1, J7.2 (Pin_2), R28.2, R29.2, R30.2, R31.2, R32.2, R33.2, R34.2, U9.13 (VDD), U9.8 (VLOGIC)
- net AGND: now also JP7.2 (B), JP8.2 (B)
- net AVDD: now also FB1.2, FB2.2, FB3.2
- net GND: now also C42.2, C43.2, C45.2, C46.2, J7.1 (Pin_1), J7.MP (MountPin), JP7.1 (A), JP8.1 (A), R27.2, TEMP1.2 (Pin_2), TEMP1.MP (MountPin), U10.17 (PGND), U10.18 (PGND), U10.25 (PGND), U9.18 (GND), U9.9 (AD0)
- net GPIO20: now also J7.3 (Pin_3), R30.1
- net GPIO21: now also J7.4 (Pin_4), R31.1
- net GPIO22: now also R28.1, U10.6 (SDA), U9.24 (SDA)
- net GPIO23: now also R29.1, U10.5 (SCL), U9.23 (SCL)
- net GPIO24: now also R32.1, U9.12 (INT)
- net GPIO25: now also R33.1, U10.7 (~{INT})
- net GPIO45: now also TP33.1
- net GPIO46: now also TP32.1
- net VUSB: now also C42.1, U10.1 (VAC), U10.24 (VBUS)
- net VBAT renamed BAT
- net BAT: now also C43.1, U10.10 (BATSNS), U10.13 (BAT), U10.14 (BAT)
- new net: C44.2, U10.21 (BTST)
- new net: TP34.1, U10.12 (~{QON})
- new net: C46.1, U10.22 (REGN)
- new net: LED6.1 (K), U10.4 (STAT)
- new net: R27.1, U10.9 (~{CE})
- new net: LED6.2 (A), R34.1
- new net BAT_SW: C44.1, L2.1, U10.19 (SW), U10.20 (SW)
- new net BAT_TEMP: TEMP1.1 (Pin_1), U10.11 (TS)
- new net VSYS: C45.1, L2.2, U10.15 (SYS), U10.16 (SYS)
- no-connect marks 2 -> 4
Other:
- note added: "DAC"
- note added: "HSTX"
- note added: "Pull-ups"
- note added: "Qwiic"
- note removed: "Connectors"
- note removed: "Temperture"
- moved on the sheet: AUDIO1, BAT1, C21, C22, C23, C24, C25, C26, C27, C28, C29, C30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

Commit message: routing complete
Parts:
- added C47, C51: 100n, Capacitor_SMD:C_0402_1005Metric_Pad0.74x0.62mm_HandSolder, symbol Device:C
- added C48: 2.2n, Capacitor_SMD:C_0402_1005Metric_Pad0.74x0.62mm_HandSolder, symbol Device:C
- added C49, C50: 1u, Capacitor_SMD:C_0402_1005Metric_Pad0.74x0.62mm_HandSolder, symbol Device:C
- added C52, C54, C55: 10u, Capacitor_SMD:C_0402_1005Metric_Pad0.74x0.62mm_HandSolder, symbol Device:C
- added Q1: SS8050, Package_TO_SOT_SMD:SOT-23, symbol Transistor_BJT:SS8050
- added R26, R36: 10k, Resistor_SMD:R_0402_1005Metric_Pad0.72x0.64mm_HandSolder, symbol Device:R
- added R35: 100, Resistor_SMD:R_0402_1005Metric_Pad0.72x0.64mm_HandSolder, symbol Device:R
- added R37: 1k, Resistor_SMD:R_0402_1005Metric_Pad0.72x0.64mm_HandSolder, symbol Device:R
- added TP35, TP36, TP37, TP38, TP39, TP40: TP, TestPoint:TestPoint_Pad_D1.0mm, symbol Connector:TestPoint
- C27, C28, C31, C32: value 470u -> 1u
- C39, C40: value 2.2u -> 2.2n
- FB1, FB2, FB3: footprint (none) -> Inductor_SMD:L_0805_2012Metric_Pad1.15x1.40mm_HandSolder
- JP6, JP7, JP8: footprint (none) -> Jumper:SolderJumper-2_P1.3mm_Bridged_Pad1.0x1.5mm
- L2: footprint (none) -> Inductor_SMD:L_6.3x6.3_H3
- NTC1: renamed from TEMP1; value temperture -> Temperture
Connections:
- net +3V3: now also C49.1, C50.1, C52.1, R35.1; no longer C27.1, C28.1, C31.1, C32.1, U6.1 (CPVDD)
- net AGND: now also C27.2, C28.2, C31.2, C32.2, C38.2, C39.1, C40.1, U6.3 (CPGND), C54.2, C55.2; no longer AUDIO1.S, C39.2, C40.2
- net AVDD: now also C27.1, C28.1, C31.1, C32.1, U6.1 (CPVDD), C54.1, C55.1
- net DAC_L: now also C39.2; no longer C39.1
- net DAC_R: now also C40.2; no longer C40.1
- net DP_BL: now also R37.1
- net DP_LED_A: now also R35.2
- net DP_LED_K: now also Q1.3 (C)
- net GND: now also AUDIO1.S, U9.1 (CLKIN), C47.2, C48.2, C49.2, C50.2, C51.2, C52.2, Q1.2 (E), R26.2, R36.2; no longer C27.2, C28.2, C31.2, C32.2, U6.3 (CPGND)
- net GPIO20: now also TP35.1
- net GPIO21: now also TP36.1
- net VSYS: now also TP39.1
- net at C38.1: now also U6.5 (VNEG)
- net at U9.10 (REGOUT): now also C47.1
- net at U9.11 (FSYNC): now also R26.1
- net at U9.20 (CPOUT): now also C48.1
- net at U10.2 (PSEL): now also TP37.1
- net at U10.23 (PMID): now also TP38.1
- net at U10.3 (PMID_GOOD): now also TP40.1
- net ~{BAT_CE}: now reaches R27.1, U10.9 (~{CE})
- net at U6.18 (LDOO): now also C51.1
- new net: Q1.1 (B), R36.1, R37.2
Other:
- moved on the sheet: BAT1, C33, C34, C37, C38, C39, C40, C45, FB1, FB2, FB3, JP6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

Commit message: Update BOM
Parts:
- BAT1, LRA1, LRA2, NTC1, SPK1, SPK2: LCSC PN (none) -> C177225
- J7: LCSC PN (none) -> C160404
- LED1, SW10, SW11, SW12, SW13, SW14, SW15, SW16, SW17, SW18, SW19, SW4, SW5, SW6, SW7, SW8, SW9, U4: now left out of the parts list
- R10, R11, R16, R17, R18, R19, R20, R21, R22, R23, R24, R25, R28, R29, R30, R31, R32, R33, R34, R37, R9: now in the parts list
Changed lines of the file:
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@@
 		(unit 1)
 		(exclude_from_sim no)
-		(in_bom no)
+		(in_bom yes)
 		(on_board yes)
 		(dnp no)
@@
 		(unit 1)
 		(exclude_from_sim no)
-		(in_bom yes)
+		(in_bom no)
 		(on_board yes)
 		(dnp no)
@@
 		(unit 1)
 		(exclude_from_sim no)
-		(in_bom no)
+		(in_bom yes)
 		(on_board yes)
 		(dnp no)
@@
 		(unit 1)
 		(exclude_from_sim no)
-		(in_bom yes)
+		(in_bom no)
 		(on_board yes)
 		(dnp no)
@@
 		(unit 1)
 		(exclude_from_sim no)
-		(in_bom yes)
+		(in_bom no)
 		(on_board yes)
 		(dnp no)
@@
 		(unit 1)
 		(exclude_from_sim no)
-		(in_bom no)
+		(in_bom yes)
 		(on_board yes)
 		(dnp no)
@@
 		(unit 1)
 		(exclude_from_sim no)
-		(in_bom no)
+		(in_bom yes)
 		(on_board yes)
 		(dnp no)
@@
 		(unit 1)
 		(exclude_from_sim no)
-		(in_bom no)
+		(in_bom yes)
 		(on_board yes)
 		(dnp no)
@@
 		(unit 1)
 		(exclude_from_sim no)
-		(in_bom no)
+		(in_bom yes)
 		(on_board yes)
 		(dnp no)
@@
 		(unit 1)
 		(exclude_from_sim no)
-		(in_bom no)
+		(in_bom yes)
 		(on_board yes)
 		(dnp no)
@@
 		(unit 1)
 		(exclude_from_sim no)
-		(in_bom no)
+		(in_bom yes)
 		(on_board yes)
 		(dnp no)
@@
 		(unit 1)
 		(exclude_from_sim no)
-		(in_bom yes)
+		(in_bom no)
 		(on_board yes)
 		(dnp no)
@@
 		(unit 1)
 		(exclude_from_sim no)
-		(in_bom yes)
+		(in_bom no)
 		(on_board yes)
 		(dnp no)
@@
 		(unit 1)
 		(exclude_from_sim no)
-		(in_bom yes)
+		(in_bom no)
 		(on_board yes)
 		(dnp no)
@@
 		(unit 1)
 		(exclude_from_sim no)
-		(in_bom yes)
+		(in_bom no)
 		(on_board yes)
 		(dnp no)
@@
 		(unit 1)
 		(exclude_from_sim no)
-		(in_bom yes)
+		(in_bom no)
 		(on_board yes)
 		(dnp no)
@@
 		(unit 1)
 		(exclude_from_sim no)
-		(in_bom yes)
+		(in_bom no)
 		(on_board yes)
 		(dnp no)
@@
 		(unit 1)
 		(exclude_from_sim no)
-		(in_bom yes)
+		(in_bom no)
 		(on_board yes)
 		(dnp no)
@@
 		(unit 1)
 		(exclude_from_sim no)
-		(in_bom no)
+		(in_bom yes)
 		(on_board yes)
 		(dnp no)
@@
 		(unit 1)
 		(exclude_from_sim no)
-		(in_bom no)
+		(in_bom yes)
 		(on_board yes)
 		(dnp no)
@@
 		(unit 1)
 		(exclude_from_sim no)
-		(in_bom yes)
+		(in_bom no)
 		(on_board yes)
 		(dnp no)
@@
 		(unit 1)
 		(exclude_from_sim no)
-		(in_bom yes)
+		(in_bom no)
 		(on_board yes)
 		(dnp no)
@@
 			)
 		)
+		(property "LCSC PN" "C177225"
+			(at 44.45 259.08 0)
+			(effects
+				(font
+					(size 1.27 1.27)
+				)
+				(hide yes)
+			)
+		)
 		(pin "2"
 		)
@@
 		(unit 1)
 		(exclude_from_sim no)
-		(in_bom no)
+		(in_bom yes)
 		(on_board yes)
 		(dnp no)
@@
 		(unit 1)
 		(exclude_from_sim no)
-		(in_bom yes)
+		(in_bom no)
 		(on_board yes)
 		(dnp no)
@@
 		(unit 1)
 		(exclude_from_sim no)
-		(in_bom yes)
+		(in_bom no)
 		(on_board yes)
 		(dnp no)
@@
 		(unit 1)
 		(exclude_from_sim no)
-		(in_bom no)
+		(in_bom yes)
 		(on_board yes)
 		(dnp no)
@@
 		(unit 1)
 		(exclude_from_sim no)
-		(in_bom no)
+		(in_bom yes)
 		(on_board yes)
 		(dnp no)
@@
 			)
 		)
+		(property "LCSC PN" "C177225"
+			(at 30.48 356.87 0)
+			(effects
+				(font
+					(size 1.27 1.27)
+				)
+				(hide yes)
+			)
+		)
 		(pin "2"
 		)
@@
 		(unit 1)
 		(exclude_from_sim no)
-		(in_bom yes)
+		(in_bom no)
 		(on_board yes)
 		(dnp no)
@@
 		(unit 1)
 		(exclude_from_sim no)
-		(in_bom yes)
+		(in_bom no)
 		(on_board yes)
 		(dnp no)
@@
 		(unit 1)
 		(exclude_from_sim no)
-		(in_bom no)
+		(in_bom yes)
 		(on_board yes)
 		(dnp no)
@@
 		(unit 1)
 		(exclude_from_sim no)
-		(in_bom no)
+		(in_bom yes)
 		(on_board yes)
 		(dnp no)
@@
 		(unit 1)
 		(exclude_from_sim no)
-		(in_bom yes)
+		(in_bom no)
 		(on_board yes)
 		(dnp no)
@@
 		(unit 1)
 		(exclude_from_sim no)
-		(in_bom no)
+		(in_bom yes)
 		(on_board yes)
 		(dnp no)
@@
 		(unit 1)
 		(exclude_from_sim no)
-		(in_bom no)
+		(in_bom yes)
 		(on_board yes)
 		(dnp no)
@@
 			)
 		)
+		(property "LCSC PN" "C177225"
+			(at 71.12 259.08 0)
+			(effects
+				(font
+					(size 1.27 1.27)
+				)
+				(hide yes)
+			)
+		)
 		(pin "2"
 		)
@@
 		(unit 1)
 		(exclude_from_sim no)
-		(in_bom no)
+		(in_bom yes)
 		(on_board yes)
 		(dnp no)
@@
 		(unit 1)
 		(exclude_from_sim no)
-		(in_bom no)
+		(in_bom yes)
 		(on_board yes)
 		(dnp no)
@@
 			)
 		)
+		(property "LCSC PN" "C177225"
+			(at 55.88 340.36 0)
+			(effects
+				(font
+					(size 1.27 1.27)
+				)
+				(hide yes)
+			)
+		)
 		(pin "2"
 		)
@@
 		(unit 1)
 		(exclude_from_sim no)
-		(in_bom no)
+		(in_bom yes)
 		(on_board yes)
 		(dnp no)
@@
 			)
 		)
+		(property "LCSC PN" "C177225"
+			(at 55.88 356.87 0)
+			(effects
+				(font
+					(size 1.27 1.27)
+				)
+				(hide yes)
+			)
+		)
 		(pin "2"
 		)
@@
 			)
 		)
+		(property "LCSC PN" "C177225"
+			(at 30.48 340.36 0)
+			(effects
+				(font
+					(size 1.27 1.27)
+				)
+				(hide yes)
+			)
+		)
 		(pin "2"
 		)
@@
 			)
 		)
+		(property "LCSC PN" "C160404"
+			(at 88.9 365.76 0)
+			(effects
+				(font
+					(size 1.27 1.27)
+				)
+				(hide yes)
+			)
+		)
 		(pin "3"
 		)
@@
 		(unit 1)
 		(exclude_from_sim no)
-		(in_bom no)
+		(in_bom yes)
 		(on_board yes)
 		(dnp no)
@@
 		(unit 1)
 		(exclude_from_sim no)
-		(in_bom yes)
+		(in_bom no)
 		(on_board yes)
 		(dnp no)

Commit message: Update schematic - Change L2 - Add NTC2 pad - Connect pins to measure voltages
Parts:
- added R38, R39, R40, R41: 10k, Resistor_SMD:R_0402_1005Metric_Pad0.72x0.64mm_HandSolder, symbol Device:R
- added TP41, TP42, TP43: TP, TestPoint:TestPoint_Pad_D1.0mm, symbol Connector:TestPoint
- AUDIO1: value AudioJack3_SwitchTR -> SJ2-35954B-SMT-TR
- L2: value 1u -> MAPM0420F-2R2M-LF; footprint Inductor_SMD:L_6.3x6.3_H3 -> Library:Inductor_SMD_L_4.9x4.4_H2
Connections:
- net +3V3: now also U5.9 (VREF), R38.1
- net BAT: now also U5.7 (VBAT)
- net GND: now also R40.2, TP42.1
- net GPIO44: now also R40.1, R41.2, TP43.1
- net VUSB: now also R39.1
- net BAT_TEMP2: now reaches U5.8 (IN)
- net BAT_TEMP2: now also R38.2, TP41.1
- net at TP37.1, U10.2 (PSEL): now also R39.2
- net BAT_TEMP renamed BAT_TEMP1
- new net VIN: R41.1
Other:
- moved on the sheet: AUDIO1, BAT1, C19, C20, C21, C22, C23, C24, C25, C26, C27, C28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
