File: pico_concole_v2_daughter_board.kicad_pcb (KiCad board)
At the start: 2 copper layers, 165.1 x 88.9 mm, 61 parts, among them J1 USB_C_Receptacle_USB2.0_16P, J2 SM03B-SRSS-TB, J3 SM03B-SRSS-TB, J4 Conn_02x12, J5 Conn_02x12, U1 PCM5102A, U2 PAM8403D, U3 RP2350_80QFN, U4 TSOP34S40F, U5 XPT2046TS

Commit message: Place components temporarily
Parts:
- removed H15, H16: M2, MountingHole:MountingHole_2.2mm_M2
- removed REF**: MountingHole_2mm, MountingHole:MountingHole_2mm
- added SW1: SW_Push, Button_Switch_THT:SM-05H-0xC-Zippy, F.Cu at (186.7, 39.4)
- added SW10: SW_Push, Button_Switch_THT:SW_PUSH_6mm_H7.3mm, F.Cu at (48.5, 89.6)
- added SW11: SW_Push, Button_Switch_THT:SW_PUSH_6mm_H7.3mm, F.Cu at (38.7, 93.0)
- added SW12: SW_Push, Button_Switch_THT:SW_PUSH_6mm_H7.3mm, F.Cu at (30.8, 89.6)
- added SW13: SW_Push, Button_Switch_THT:SW_PUSH_6mm_H7.3mm, F.Cu at (53.9, 31.4)
- added SW14: SW_Push, Button_Switch_THT:SW_PUSH_6mm_H7.3mm, F.Cu at (162.0, 35.9)
- added SW15: SW_Push, Button_Switch_THT:SW_PUSH_6mm_H7.3mm, F.Cu at (78.0, 28.2)
- added SW16: SW_Push, Button_Switch_THT:SW_PUSH_6mm_H7.3mm, F.Cu at (137.9, 32.7)
- added SW17: SW_Push, Button_Switch_SMD:SW_SPST_PTS810, F.Cu at (108.0, 109.2)
- added SW2: SW_Push, Button_Switch_THT:SM-05H-0xD-Zippy, B.Cu at (182.5, 39.4)
- added SW3: SW_Push, Button_Switch_THT:SM-05H-0xC-Zippy, B.Cu at (33.4, 39.4)
- added SW4: SW_Push, Button_Switch_THT:SM-05H-0xD-Zippy, F.Cu at (29.2, 39.4)
- added SW5: SW_Push, Button_Switch_THT:SW_PUSH_6mm_H7.3mm, F.Cu at (170.7, 42.8)
- added SW6: SW_Push, Button_Switch_THT:SW_PUSH_6mm_H7.3mm, F.Cu at (180.6, 57.2)
- added SW7: SW_Push, Button_Switch_THT:SW_PUSH_6mm_H7.3mm, F.Cu at (170.7, 60.6)
- added SW8: SW_Push, Button_Switch_THT:SW_PUSH_6mm_H7.3mm, F.Cu at (162.8, 57.2)
- added SW9: SW_Push, Button_Switch_THT:SW_PUSH_6mm_H7.3mm, F.Cu at (38.7, 75.2)
- moved H12 201.9 mm to (29.2, 97.8)
- moved H9 199.5 mm to (29.2, 43.2)
- moved H14 193.3 mm to (41.9, 69.8)
- moved H8 154.3 mm to (58.4, 116.8)
- moved H5 141.0 mm to (64.8, 29.2)
- moved H7 111.4 mm to (157.5, 116.8)
- moved R4 109.2 mm to (113.5, 31.2), turned to 90 degrees
- moved H6 108.0 mm to (151.1, 29.2)
- moved H13 64.3 mm to (174.0, 69.8)
- moved JP1 62.6 mm to (207.3, 39.4)
- moved JP2 62.6 mm to (207.3, 41.9)
- moved JP3 62.6 mm to (207.3, 44.5)
- moved JP4 62.6 mm to (207.3, 47.0)
- moved R5 62.6 mm to (199.7, 39.4)
- moved R6 62.6 mm to (199.7, 41.9)
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Routing:
- net GND: vias 0 -> 78
- added copper zone on B.Cu, net GND
- added copper zone on F.Cu, net GND
Other:
- board size 165.1 x 88.9 mm -> 165.1 x 95.2 mm
- board text added: "+"
- board text added: "4.0{dblquote} Display with touch panel"
- board text added: "A"
- board text added: "B"
- board text added: "Battery"
- board text added: "Designed by"
- board text added: "L"
- board text added: "L Stick"
- board text added: "LRA module (23*10mm)"
- board text added: "POWER"
- board text added: "R"
- board text added: "R Stick"
- board text added: "RESET"
- board text added: "RP2350A Main board"
- board text added: "SELECT"
- board text added: "START"
- board text added: "SUB1"
- board text added: "SUB2"
- board text added: "X"
- board text added: "Y"
- board text added: "ZL"
- board text added: "ZR"
- board text removed: "4.0' DISPLAY +"
- board text removed: "LRA module"

Commit message: Place components temporarily
Parts:
- added D1: D_Small, Diode_SMD:D_0805_2012Metric_Pad1.15x1.40mm_HandSolder, F.Cu at (99.7, 129.5)
- added D10: D_Small, Diode_SMD:D_0805_2012Metric_Pad1.15x1.40mm_HandSolder, B.Cu at (47.5, 86.4)
- added D11: D_Small, Diode_SMD:D_0805_2012Metric_Pad1.15x1.40mm_HandSolder, B.Cu at (41.9, 91.9)
- added D12: D_Small, Diode_SMD:D_0805_2012Metric_Pad1.15x1.40mm_HandSolder, B.Cu at (36.3, 86.4)
- added D13: D_Small, Diode_SMD:D_0805_2012Metric_Pad1.15x1.40mm_HandSolder, F.Cu at (124.7, 130.6)
- added D14: D_Small, Diode_SMD:D_0805_2012Metric_Pad1.15x1.40mm_HandSolder, F.Cu at (124.7, 133.6)
- added D15: D_Small, Diode_SMD:D_0805_2012Metric_Pad1.15x1.40mm_HandSolder, F.Cu at (124.7, 136.7)
- added D16: D_Small, Diode_SMD:D_0805_2012Metric_Pad1.15x1.40mm_HandSolder, F.Cu at (124.7, 139.7)
- added D2: D_Small, Diode_SMD:D_0805_2012Metric_Pad1.15x1.40mm_HandSolder, F.Cu at (99.7, 132.6)
- added D3: D_Small, Diode_SMD:D_0805_2012Metric_Pad1.15x1.40mm_HandSolder, F.Cu at (99.7, 135.6)
- added D4: D_Small, Diode_SMD:D_0805_2012Metric_Pad1.15x1.40mm_HandSolder, F.Cu at (99.7, 138.7)
- added D5: D_Small, Diode_SMD:D_0805_2012Metric_Pad1.15x1.40mm_HandSolder, B.Cu at (174.0, 48.3)
- added D6: D_Small, Diode_SMD:D_0805_2012Metric_Pad1.15x1.40mm_HandSolder, B.Cu at (179.6, 54.0)
- added D7: D_Small, Diode_SMD:D_0805_2012Metric_Pad1.15x1.40mm_HandSolder, B.Cu at (174.0, 59.4)
- added D8: D_Small, Diode_SMD:D_0805_2012Metric_Pad1.15x1.40mm_HandSolder, B.Cu at (168.4, 54.0)
- added D9: D_Small, Diode_SMD:D_0805_2012Metric_Pad1.15x1.40mm_HandSolder, B.Cu at (41.9, 80.8)
- added JOY1: Joy1, Connector_FFC-FPC:TE_0-1734839-5_1x05-1MP_P0.5mm_Horizontal, B.Cu at (29.8, 75.8)
- added JOY2: Joy2, Connector_FFC-FPC:TE_0-1734839-5_1x05-1MP_P0.5mm_Horizontal, B.Cu at (186.1, 64.5)
- moved LRA1 16.0 mm to (50.2, 101.0), turned to 90 degrees
- moved LRA2 16.0 mm to (165.7, 101.0), turned to -90 degrees
- moved SW10 7.91 mm to (53.0, 83.1), turned to -90 degrees
- moved SW11 7.91 mm to (45.2, 97.5), turned to 180 degrees
- moved SW6 7.91 mm to (185.1, 50.7), turned to -90 degrees
- moved SW7 7.91 mm to (177.2, 65.1), turned to 180 degrees
- moved H11 3.24 mm to (183.5, 98.4)
- moved H12 3.24 mm to (32.4, 98.4)
- moved H9 0.90 mm to (29.8, 43.8)
- moved H10 0.90 mm to (186.1, 43.8)
Routing:
- net /Daughterboard/BTN_H2: track 0.00 -> 26.0 mm
- net /Daughterboard/BTN_H3: track 0.00 -> 25.8 mm
- net /Daughterboard/BTN_V4: track 0.00 -> 13.0 mm
- net /Daughterboard/BTN_V3: track 0.00 -> 13.0 mm
- net /Daughterboard/BTN_V2: track 0.00 -> 13.0 mm
- net /Daughterboard/BTN_V1: track 0.00 -> 13.0 mm
- net Net-(D9-A): track 0.00 -> 6.50 mm
- net Net-(D8-A): track 0.00 -> 6.50 mm
- net Net-(D7-A): track 0.00 -> 6.50 mm
- net Net-(D6-A): track 0.00 -> 6.50 mm
- net Net-(D5-A): track 0.00 -> 6.50 mm
- net Net-(D12-A): track 0.00 -> 6.50 mm
- net Net-(D11-A): track 0.00 -> 6.50 mm
- net Net-(D10-A): track 0.00 -> 6.50 mm
- net Net-(R3-Pad1): track 0.00 -> 4.15 mm
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Other:
- outline, holes or cut-outs redrawn

Commit message: v2.0.0 WIP
Parts:
- removed H13, H14: M2, MountingHole:MountingHole_2.2mm_M2
- added C1: 1u, Capacitor_SMD:C_0402_1005Metric_Pad0.74x0.62mm_HandSolder, B.Cu at (134.0, 89.5)
- added C2: 470n, Capacitor_SMD:C_0402_1005Metric_Pad0.74x0.62mm_HandSolder, B.Cu at (135.9, 90.8)
- added C3: 470n, Capacitor_SMD:C_0402_1005Metric_Pad0.74x0.62mm_HandSolder, B.Cu at (135.9, 81.9)
- added C4: 470u, Capacitor_SMD:C_0402_1005Metric_Pad0.74x0.62mm_HandSolder, B.Cu at (137.8, 91.4)
- added C5: 470u, Capacitor_SMD:C_0402_1005Metric_Pad0.74x0.62mm_HandSolder, B.Cu at (140.3, 81.3)
- added C6: 1u, Capacitor_SMD:C_0402_1005Metric_Pad0.74x0.62mm_HandSolder, B.Cu at (140.3, 91.4)
- added C7: 1u, Capacitor_SMD:C_0402_1005Metric_Pad0.74x0.62mm_HandSolder, B.Cu at (137.8, 81.3)
- added R10: 1k, Resistor_SMD:R_0603_1608Metric_Pad0.98x0.95mm_HandSolder, B.Cu at (139.1, 80.6)
- added R9: 1k, Resistor_SMD:R_0603_1608Metric_Pad0.98x0.95mm_HandSolder, B.Cu at (139.1, 92.1)
- D1, D13, D14, D15, D16, D2, D3, D4: moved to B.Cu
- moved D2 145.0 mm to (138.7, -7.12), turned to 180 degrees
- moved D3 145.0 mm to (138.7, -4.08), turned to 180 degrees
- moved D4 145.0 mm to (138.7, -1.04), turned to 180 degrees
- moved D1 133.5 mm to (138.7, 1.91), turned to 180 degrees
- moved SW15 86.7 mm to (54.9, 111.8), turned to 90 degrees
- moved SW16 76.2 mm to (161.0, 105.3), turned to -90 degrees
- moved BAT1 25.5 mm to (137.8, 41.9), turned to -90 degrees
- moved U5 21.9 mm to (87.6, 84.5), turned to 180 degrees
- moved D13 11.7 mm to (113.0, 130.2), turned to 180 degrees
- moved D14 11.7 mm to (113.0, 133.2), turned to 180 degrees
- moved D15 11.7 mm to (113.0, 136.3), turned to 180 degrees
- moved D16 11.7 mm to (113.0, 139.3), turned to 180 degrees
- moved SPK1 7.85 mm to (81.3, 101.0)
- moved SPK2 7.85 mm to (134.6, 101.0)
- moved SW14 6.22 mm to (161.0, 29.8), turned to -90 degrees
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Connections:
- net /Daughterboard/Joy1_X renamed /Daughterboard/GPIO40_ADC0
- net /Daughterboard/Joy1_Y renamed /Daughterboard/GPIO41_ADC1
- net /Daughterboard/Joy2_X renamed /Daughterboard/GPIO42_ADC2
- net /Daughterboard/Joy2_Y renamed /Daughterboard/GPIO43_ADC3
- D1 pad 1: /Daughterboard/BTN_H1 -> /Daughterboard/GPIO32
- D10 pad 1: /Daughterboard/BTN_H3 -> /Daughterboard/GPIO34
- D11 pad 1: /Daughterboard/BTN_H3 -> /Daughterboard/GPIO34
- D12 pad 1: /Daughterboard/BTN_H3 -> /Daughterboard/GPIO34
- D13 pad 1: /Daughterboard/BTN_H4 -> /Daughterboard/GPIO35
- D14 pad 1: /Daughterboard/BTN_H4 -> /Daughterboard/GPIO35
- D15 pad 1: /Daughterboard/BTN_H4 -> /Daughterboard/GPIO35
- D16 pad 1: /Daughterboard/BTN_H4 -> /Daughterboard/GPIO35
- D2 pad 1: /Daughterboard/BTN_H1 -> /Daughterboard/GPIO32
- D3 pad 1: /Daughterboard/BTN_H1 -> /Daughterboard/GPIO32
- D4 pad 1: /Daughterboard/BTN_H1 -> /Daughterboard/GPIO32
- D5 pad 1: /Daughterboard/BTN_H2 -> /Daughterboard/GPIO33
- D6 pad 1: /Daughterboard/BTN_H2 -> /Daughterboard/GPIO33
- D7 pad 1: /Daughterboard/BTN_H2 -> /Daughterboard/GPIO33
- D8 pad 1: /Daughterboard/BTN_H2 -> /Daughterboard/GPIO33
- D9 pad 1: /Daughterboard/BTN_H3 -> /Daughterboard/GPIO34
- DP1 pad 1: unconnected-(DP1-Pin_1-Pad1) -> /Daughterboard/TP_X-
- DP1 pad 10: unconnected-(DP1-Pin_10-Pad10) -> /Daughterboard/MAIN_GPIO18
- DP1 pad 11: unconnected-(DP1-Pin_11-Pad11) -> /Daughterboard/MAIN_GPIO17
- DP1 pad 12: unconnected-(DP1-Pin_12-Pad12) -> +3V3
- DP1 pad 13: unconnected-(DP1-Pin_13-Pad13) -> /Daughterboard/MAIN_GPIO16
- DP1 pad 14: unconnected-(DP1-Pin_14-Pad14) -> /Daughterboard/DP_MISO
- DP1 pad 15: unconnected-(DP1-Pin_15-Pad15) -> /Daughterboard/MAIN_GPIO15
- DP1 pad 2: unconnected-(DP1-Pin_2-Pad2) -> /Daughterboard/TP_Y+
- DP1 pad 3: unconnected-(DP1-Pin_3-Pad3) -> /Daughterboard/TP_X+
- DP1 pad 4: unconnected-(DP1-Pin_4-Pad4) -> /Daughterboard/TP_Y-
- DP1 pad 9: unconnected-(DP1-Pin_9-Pad9) -> /Daughterboard/MAIN_GPIO14
- JOY1 pad 3: /Daughterboard/Joy1_BTN -> /Daughterboard/GPIO26
- JOY2 pad 3: /Daughterboard/Joy2_BTN -> /Daughterboard/GPIO27
- SW1 pad 1: /Daughterboard/BTN_V1 -> /Daughterboard/GPIO28
- SW10 pad 1: /Daughterboard/BTN_V2 -> /Daughterboard/GPIO29
- SW11 pad 1: /Daughterboard/BTN_V3 -> /Daughterboard/GPIO30
- SW12 pad 1: /Daughterboard/BTN_V4 -> /Daughterboard/GPIO31
- SW13 pad 1: /Daughterboard/BTN_V1 -> /Daughterboard/GPIO28
- SW14 pad 1: /Daughterboard/BTN_V2 -> /Daughterboard/GPIO29
- SW15 pad 1: /Daughterboard/BTN_V3 -> /Daughterboard/GPIO30
- SW16 pad 1: /Daughterboard/BTN_V4 -> /Daughterboard/GPIO31
- SW2 pad 1: /Daughterboard/BTN_V2 -> /Daughterboard/GPIO29
- SW3 pad 1: /Daughterboard/BTN_V3 -> /Daughterboard/GPIO30
- SW4 pad 1: /Daughterboard/BTN_V4 -> /Daughterboard/GPIO31
- SW5 pad 1: /Daughterboard/BTN_V1 -> /Daughterboard/GPIO28
- SW6 pad 1: /Daughterboard/BTN_V2 -> /Daughterboard/GPIO29
- SW7 pad 1: /Daughterboard/BTN_V3 -> /Daughterboard/GPIO30
- SW8 pad 1: /Daughterboard/BTN_V4 -> /Daughterboard/GPIO31
- SW9 pad 1: /Daughterboard/BTN_V1 -> /Daughterboard/GPIO28
- U1 pad 13: /Daughterboard/I2S_SCK -> /Daughterboard/GPIO37
- U1 pad 14: /Daughterboard/I2S_DATA -> /Daughterboard/GPIO36
- U1 pad 15: /Daughterboard/I2S_LRCK -> /Daughterboard/GPIO38
- U1 pad 17: /Daughterboard/~{AMP_MUTE} -> /Daughterboard/GPIO39
- U2 pad 10: /Daughterboard/SPK_R -> Net-(U2-INR)
- U2 pad 11: unconnected-(U2-GND-Pad11) -> GNDA
- U2 pad 12: unconnected-(U2-~{SHDN}-Pad12) -> Net-(U2-~{SHDN})
- U2 pad 13: Net-(U2-PVDD-Pad13) -> VIN
- U2 pad 15: Net-(U2-PGND-Pad15) -> GNDA
- U2 pad 2: Net-(U2-PGND-Pad15) -> GNDA
- U2 pad 4: Net-(U2-PVDD-Pad13) -> VIN
- U2 pad 5: unconnected-(U2-~{MUTE}-Pad5) -> Net-(U2-~{MUTE})
- U2 pad 6: unconnected-(U2-VDD-Pad6) -> VIN
- U2 pad 7: /Daughterboard/SPK_L -> Net-(U2-INL)
- U2 pad 8: unconnected-(U2-VREF-Pad8) -> Net-(U2-VREF)
- U3 pad 1: /Daughterboard/GPIO4 -> /Daughterboard/MAIN_GPIO13
- U3 pad 2: /Daughterboard/GPIO5 -> /Daughterboard/MAIN_GPIO12
- U5 pad 11: /Daughterboard/~{TOUCH_IRQ} -> /Daughterboard/MAIN_GPIO24
- U5 pad 12: /Daughterboard/TOUCH_MISO -> /Daughterboard/MAIN_GPIO20
- U5 pad 14: /Daughterboard/TOUCH_MOSI -> /Daughterboard/MAIN_GPIO23
- U5 pad 15: /Daughterboard/~{TOUCH_CS} -> /Daughterboard/MAIN_GPIO21
- U5 pad 16: /Daughterboard/TOUCH_SCK -> /Daughterboard/MAIN_GPIO22
Routing:
- net /Daughterboard/GPIO33: track 0.00 -> 34.7 mm
- net /Daughterboard/GPIO34: track 0.00 -> 34.5 mm
- net /Daughterboard/BTN_H2: track 26.0 -> 0.00 mm
- net /Daughterboard/BTN_H3: track 25.8 -> 0.00 mm
- net /Daughterboard/GPIO31: track 0.00 -> 13.0 mm
- net /Daughterboard/GPIO30: track 0.00 -> 13.0 mm
- net /Daughterboard/GPIO29: track 0.00 -> 13.0 mm
- net /Daughterboard/GPIO28: track 0.00 -> 13.0 mm
- net /Daughterboard/BTN_V4: track 13.0 -> 0.00 mm
- net /Daughterboard/BTN_V3: track 13.0 -> 0.00 mm
- net /Daughterboard/BTN_V2: track 13.0 -> 0.00 mm
- net /Daughterboard/BTN_V1: track 13.0 -> 0.00 mm
Other:
- outline, holes or cut-outs redrawn
- board text added: "DEBUG"
- board text added: "LOG"
- board text added: "USB"
- board text added: "USER"
- board text added: "microSD"

Commit message: v2.0.0 WIP
Parts:
- added C10: 1u, Capacitor_SMD:C_0402_1005Metric_Pad0.74x0.62mm_HandSolder, B.Cu at (66.6, 96.0)
- added C11: 470u, Capacitor_SMD:C_0402_1005Metric_Pad0.74x0.62mm_HandSolder, B.Cu at (66.6, 98.0)
- added C12: 470u, Capacitor_SMD:C_0402_1005Metric_Pad0.74x0.62mm_HandSolder, B.Cu at (66.6, 100.0)
- added C13: 1u, Capacitor_SMD:C_0402_1005Metric_Pad0.74x0.62mm_HandSolder, B.Cu at (66.6, 101.9)
- added C14: 1u, Capacitor_SMD:C_0402_1005Metric_Pad0.74x0.62mm_HandSolder, B.Cu at (66.6, 103.9)
- added C8: 470n, Capacitor_SMD:C_0402_1005Metric_Pad0.74x0.62mm_HandSolder, B.Cu at (66.6, 92.1)
- added C9: 470n, Capacitor_SMD:C_0402_1005Metric_Pad0.74x0.62mm_HandSolder, B.Cu at (66.6, 94.0)
- added R11: 1k, Resistor_SMD:R_0603_1608Metric_Pad0.98x0.95mm_HandSolder, B.Cu at (65.4, 97.2)
- added R12: 1k, Resistor_SMD:R_0603_1608Metric_Pad0.98x0.95mm_HandSolder, B.Cu at (65.4, 99.7)
- added TP11: TP, TestPoint:TestPoint_Pad_1.0x1.0mm, B.Cu at (82.4, 136.1)
- added TP12: TP, TestPoint:TestPoint_Pad_1.0x1.0mm, B.Cu at (84.5, 134.9)
- added TP13: TP, TestPoint:TestPoint_Pad_1.0x1.0mm, B.Cu at (82.4, 134.1)
- added TP14: TP, TestPoint:TestPoint_Pad_1.0x1.0mm, B.Cu at (84.5, 132.8)
- added TP15: TP, TestPoint:TestPoint_Pad_1.0x1.0mm, B.Cu at (82.4, 132.1)
- added TP16: TP, TestPoint:TestPoint_Pad_1.0x1.0mm, B.Cu at (84.5, 130.8)
- added TP17: TP, TestPoint:TestPoint_Pad_1.0x1.0mm, B.Cu at (82.4, 130.0)
- added TP18: TP, TestPoint:TestPoint_Pad_1.0x1.0mm, B.Cu at (84.5, 128.8)
- added TP19: TP, TestPoint:TestPoint_Pad_1.0x1.0mm, B.Cu at (84.5, 140.8)
- added TP20: TP, TestPoint:TestPoint_Pad_1.0x1.0mm, B.Cu at (82.4, 140.8)
- added TP21: TP, TestPoint:TestPoint_Pad_1.0x1.0mm, B.Cu at (63.5, 40.4)
- added TP22: TP, TestPoint:TestPoint_Pad_1.0x1.0mm, B.Cu at (63.5, 42.4)
- added TP23: TP, TestPoint:TestPoint_Pad_1.0x1.0mm, B.Cu at (107.3, 133.3)
- added U6: PAM8403D, Package_SO:SOIC-16_3.9x9.9mm_P1.27mm, B.Cu at (66.7, 98.4)
- moved R8 79.4 mm to (90.8, 107.3), turned to 180 degrees
- moved U4 34.2 mm to (107.3, 56.5), turned to 0 degrees
- moved R10 23.4 mm to (154.3, 98.4), turned to 180 degrees
- moved C5 22.7 mm to (153.7, 99.7), turned to 0 degrees
- moved C7 22.5 mm to (153.7, 97.2), turned to 180 degrees
- moved C2 21.7 mm to (153.0, 95.2), turned to -90 degrees
- moved U5 15.5 mm to (148.6, 99.1), turned to 0 degrees
- moved C3 12.0 mm to (145.4, 93.3), turned to 180 degrees
- moved C1 9.38 mm to (144.1, 95.2), turned to -90 degrees
- moved C6 8.84 mm to (143.5, 99.7), turned to 180 degrees
- moved C4 8.08 mm to (143.5, 97.2), turned to 180 degrees
- moved R9 7.41 mm to (142.9, 98.4), turned to 0 degrees
- moved LED1 6.25 mm to (92.7, 34.3)
- moved LED4 6.25 mm to (123.2, 34.3)
- moved SW5 6.22 mm to (60.4, 33.4), turned to 180 degrees
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- renumbered C2 to C1, C3 to C2, C1 to C3, D7 to D10, D15 to D12, D4 to D13, D8 to D14, D12 to D15, D5 to D2, D9 to D3, D13 to D4, D2 to D5, D10 to D7, D14 to D8, D3 to D9, H4 to H10, H8 to H11, H5 to H2, H9 to H3, H2 to H4, H6 to H5, H10 to H6, H3 to H7, H7 to H8, H11 to H9, J5 to J4, J4 to J5, R5 to R3, R6 to R4, R7 to R5, R8 to R6, R3 to R7, R4 to R8, SW17 to SW1, SW3 to SW10, SW7 to SW11, SW11 to SW12, SW15 to SW13, SW4 to SW14, SW8 to SW15, SW12 to SW16, SW16 to SW17, SW1 to SW2, SW5 to SW3, SW9 to SW4, SW13 to SW5, SW2 to SW6, SW6 to SW7, SW10 to SW8, SW14 to SW9, TP9 to TP1, TP1 to TP2, TP5 to TP4, TP7 to TP5, TP2 to TP6, TP4 to TP7, TP6 to TP8, TP8 to TP9, U3 to U1, U1 to U2, U4 to U3, U5 to U4, U2 to U5
Connections:
- net /Southbridge/GPIO44_ADC4 renamed /Daughterboard/GPIO44
- net /Southbridge/GPIO45_ADC5 renamed /Daughterboard/GPIO45
- net /Southbridge/GPIO46_ADC6 renamed /Daughterboard/GPIO46
- C1 pad 1: /Daughterboard/SPK_L -> /Daughterboard/SPK_R
- C2 pad 1: /Daughterboard/SPK_R -> /Daughterboard/GPIO10
- DP1 pad 1: /Daughterboard/TP_X- -> +3V3
- DP1 pad 10: /Daughterboard/MAIN_GPIO18 -> GND
- DP1 pad 11: /Daughterboard/MAIN_GPIO17 -> GND
- DP1 pad 12: +3V3 -> GND
- DP1 pad 13: /Daughterboard/MAIN_GPIO16 -> GND
- DP1 pad 14: /Daughterboard/DP_MISO -> GND
- DP1 pad 15: /Daughterboard/MAIN_GPIO15 -> GND
- DP1 pad 2: /Daughterboard/TP_Y+ -> +3V3
- DP1 pad 26: GND -> /Daughterboard/MAIN_GPIO15
- DP1 pad 27: GND -> /Daughterboard/DP_MISO
- DP1 pad 28: GND -> /Daughterboard/MAIN_GPIO16
- DP1 pad 29: GND -> +3V3
- DP1 pad 3: /Daughterboard/TP_X+ -> +3V3
- DP1 pad 30: GND -> /Daughterboard/MAIN_GPIO17
- DP1 pad 31: GND -> /Daughterboard/MAIN_GPIO18
- DP1 pad 32: GND -> /Daughterboard/MAIN_GPIO14
- DP1 pad 34: Net-(DP1-Pin_34) -> +3V3
- DP1 pad 35: Net-(DP1-Pin_34) -> +3V3
- DP1 pad 36: Net-(DP1-Pin_34) -> GND
- DP1 pad 37: GND -> /Daughterboard/TP_Y-
- DP1 pad 38: +3V3 -> /Daughterboard/TP_X+
- DP1 pad 39: +3V3 -> /Daughterboard/TP_Y+
- DP1 pad 4: /Daughterboard/TP_Y- -> GND
- DP1 pad 40: +3V3 -> /Daughterboard/TP_X-
- DP1 pad 5: GND -> Net-(DP1-Pin_5)
- DP1 pad 6: Net-(DP1-Pin_6) -> Net-(DP1-Pin_5)
- DP1 pad 7: Net-(DP1-Pin_6) -> Net-(DP1-Pin_5)
- DP1 pad 9: /Daughterboard/MAIN_GPIO14 -> GND
- JOY1 pad 2: /Daughterboard/GPIO41_ADC1 -> /Daughterboard/GPIO41
- JOY1 pad 5: /Daughterboard/GPIO40_ADC0 -> /Daughterboard/GPIO40
- JOY2 pad 2: /Daughterboard/GPIO43_ADC3 -> /Daughterboard/GPIO43
- JOY2 pad 5: /Daughterboard/GPIO42_ADC2 -> /Daughterboard/GPIO42
- U1 pad 49: /Southbridge/GPIO40_ADC0 -> /Daughterboard/GPIO40
- U1 pad 52: /Southbridge/GPIO41_ADC1 -> /Daughterboard/GPIO41
- U1 pad 53: /Southbridge/GPIO42_ADC2 -> /Daughterboard/GPIO42
- U1 pad 54: /Southbridge/GPIO43_ADC3 -> /Daughterboard/GPIO43
- U1 pad 58: /Southbridge/GPIO47_ADC7 -> /Daughterboard/GPIO47
- U5 pad 1: /Daughterboard/SPK_L+ -> /Daughterboard/SPK_R+
- U5 pad 14: /Daughterboard/SPK_R- -> /Daughterboard/LRA_R-
- U5 pad 16: /Daughterboard/SPK_R+ -> /Daughterboard/LRA_R+
- U5 pad 3: /Daughterboard/SPK_L- -> /Daughterboard/SPK_R-
Routing:
- net (no net): track 0.00 -> 359.3 mm
- net /Daughterboard/GPIO42: track 0.00 -> 32.2 mm, vias 0 -> 1
- net /Daughterboard/GPIO43: track 0.00 -> 27.9 mm, vias 0 -> 1
- net /Daughterboard/GPIO40: track 0.00 -> 19.0 mm, vias 0 -> 1
- net /Daughterboard/GPIO41: track 0.00 -> 18.6 mm, vias 0 -> 1
- net /Daughterboard/GPIO26: track 0.00 -> 1.41 mm, vias 0 -> 1
- net GND: vias 93 -> 95
- net /Daughterboard/GPIO27: vias 0 -> 1
Other:
- outline, holes or cut-outs redrawn
