File: pico_concole_v2_daughter_board.kicad_pcb (KiCad board)
At the start: 2 copper layers, 165.1 x 95.2 mm, 169 parts, among them J1 SM03B-SRSS-TB, J2 SM03B-SRSS-TB, J3 USB_C_Receptacle_USB2.0_16P, J4 Conn_02x12, J5 Conn_02x12, J6 Conn_01x10_MountingPin, SW1 SW_Push, SW10 SW_Push, SW11 SW_Push, SW12 SW_Push, SW13 SW_Push, SW14 SW_Push, SW15 SW_Push, SW16 SW_Push, SW17 SW_Push, SW18 SW_Push, SW19 SW_Push, SW2 SW_Push, SW3 SW_Push, SW4 SW_Push, SW5 SW_Push, SW6 SW_Push, SW7 SW_Push, SW8 SW_Push, SW9 SW_Push, U1 USBLC6-2SC6, U2 RP2350_80QFN, U3 W25Q16JVSS, U4 TSOP34S40F, U5 XPT2046TS, U6 PCM5102A, U7 PAM8403D, U8 PAM8403D, Y1 ABM8-272-T3

Commit message: V2.0.0 WIP
Parts:
- added C35: 1u, Capacitor_SMD:C_0402_1005Metric_Pad0.74x0.62mm_HandSolder, B.Cu at (111.1, 61.0)
- added C36: 1u, Capacitor_SMD:C_0402_1005Metric_Pad0.74x0.62mm_HandSolder, B.Cu at (111.1, 53.3)
- added C37: 2.2u, Capacitor_SMD:C_0402_1005Metric_Pad0.74x0.62mm_HandSolder, B.Cu at (131.0, 89.5)
- added C38: 2.2u, Capacitor_SMD:C_0402_1005Metric_Pad0.74x0.62mm_HandSolder, B.Cu at (128.9, 82.8)
- added C39: 2.2u, Capacitor_SMD:C_0402_1005Metric_Pad0.74x0.62mm_HandSolder, B.Cu at (127.6, 88.3)
- added C40: 2.2u, Capacitor_SMD:C_0402_1005Metric_Pad0.74x0.62mm_HandSolder, B.Cu at (127.6, 85.7)
- added C41: 1u, Capacitor_SMD:C_0402_1005Metric_Pad0.74x0.62mm_HandSolder, B.Cu at (84.5, 87.6)
- added R24: 470, Resistor_SMD:R_0402_1005Metric_Pad0.72x0.64mm_HandSolder, B.Cu at (129.4, 87.6)
- added R25: 470, Resistor_SMD:R_0402_1005Metric_Pad0.72x0.64mm_HandSolder, B.Cu at (129.4, 86.4)
- added R26: 0, Resistor_SMD:R_0402_1005Metric_Pad0.72x0.64mm_HandSolder, F.Cu at (78.1, 17.8)
- R18, R19: value 1k -> 100k
- moved D16 138.2 mm to (45.5, 16.1)
- moved D3 122.3 mm to (174.0, 59.1), turned to -90 degrees
- moved D4 116.9 mm to (168.9, 54.0)
- moved D15 34.4 mm to (54.6, 129.5)
- moved D8 29.3 mm to (161.9, 82.5), turned to -90 degrees
- moved D7 23.3 mm to (162.1, 39.4), turned to 90 degrees
- moved D6 21.4 mm to (164.0, 39.4), turned to 90 degrees
- moved D14 21.4 mm to (158.4, 16.5)
- moved D2 18.7 mm to (179.1, 54.0)
- moved D1 12.7 mm to (174.0, 48.9), turned to 90 degrees
- moved D5 12.0 mm to (165.9, 39.4)
- moved SW18 7.91 mm to (59.4, 105.3), turned to -90 degrees
- moved SW19 7.91 mm to (156.5, 111.8), turned to 90 degrees
- moved U6 4.19 mm to (136.1, 87.6)
- moved D13 1.91 mm to (51.4, 37.5)
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Connections:
- AUDIO1 pad R: /Daughterboard/AMP_L -> /Daughterboard/DAC_L
- AUDIO1 pad S: GND -> AGND
- AUDIO1 pad T: /Daughterboard/AMP_R -> /Daughterboard/DAC_R
- D1 pad 1: /Daughterboard/GPIO32 -> /Daughterboard/BTN_H1
- D10 pad 1: /Daughterboard/GPIO34 -> /Daughterboard/BTN_H3
- D11 pad 1: /Daughterboard/GPIO34 -> /Daughterboard/BTN_H3
- D12 pad 1: /Daughterboard/GPIO34 -> /Daughterboard/BTN_H3
- D13 pad 1: /Daughterboard/GPIO35 -> /Daughterboard/BTN_H4
- D14 pad 1: /Daughterboard/GPIO35 -> /Daughterboard/BTN_H4
- D15 pad 1: /Daughterboard/GPIO35 -> /Daughterboard/BTN_H4
- D16 pad 1: /Daughterboard/GPIO35 -> /Daughterboard/BTN_H4
- D2 pad 1: /Daughterboard/GPIO32 -> /Daughterboard/BTN_H1
- D3 pad 1: /Daughterboard/GPIO32 -> /Daughterboard/BTN_H1
- D4 pad 1: /Daughterboard/GPIO32 -> /Daughterboard/BTN_H1
- D5 pad 1: /Daughterboard/GPIO33 -> /Daughterboard/BTN_H2
- D6 pad 1: /Daughterboard/GPIO33 -> /Daughterboard/BTN_H2
- D7 pad 1: /Daughterboard/GPIO33 -> /Daughterboard/BTN_H2
- D8 pad 1: /Daughterboard/GPIO33 -> /Daughterboard/BTN_H2
- D9 pad 1: /Daughterboard/GPIO34 -> /Daughterboard/BTN_H3
- R11 pad 1: /Daughterboard/MAIN_GPIO25 -> /Daughterboard/~{SB_RUN}
- R11 pad 2: /Daughterboard/~{SB_RUN} -> /Daughterboard/MAIN_GPIO25
- SW10 pad 1: /Daughterboard/GPIO30 -> /Daughterboard/BTN_V3
- SW10 pad 2: Net-(D7-A) -> Net-(D3-A)
- SW11 pad 1: /Daughterboard/GPIO31 -> /Daughterboard/BTN_V4
- SW11 pad 2: Net-(D8-A) -> Net-(D4-A)
- SW12 pad 1: /Daughterboard/GPIO28 -> /Daughterboard/BTN_V1
- SW13 pad 1: /Daughterboard/GPIO29 -> /Daughterboard/BTN_V2
- SW14 pad 1: /Daughterboard/GPIO30 -> /Daughterboard/BTN_V3
- SW15 pad 1: /Daughterboard/GPIO31 -> /Daughterboard/BTN_V4
- SW16 pad 1: /Daughterboard/GPIO28 -> /Daughterboard/BTN_V1
- SW17 pad 1: /Daughterboard/GPIO29 -> /Daughterboard/BTN_V3
- SW17 pad 2: Net-(D14-A) -> Net-(D7-A)
- SW18 pad 1: /Daughterboard/GPIO30 -> /Daughterboard/BTN_V3
- SW19 pad 1: /Daughterboard/GPIO31 -> /Daughterboard/BTN_V4
- SW19 pad 2: Net-(D16-A) -> Net-(D8-A)
- SW4 pad 1: /Daughterboard/GPIO28 -> /Daughterboard/BTN_V2
- SW4 pad 2: Net-(D1-A) -> Net-(D6-A)
- SW5 pad 1: /Daughterboard/GPIO29 -> /Daughterboard/BTN_V1
- SW5 pad 2: Net-(D2-A) -> Net-(D5-A)
- SW6 pad 1: /Daughterboard/GPIO30 -> /Daughterboard/BTN_V2
- SW6 pad 2: Net-(D3-A) -> Net-(D14-A)
- SW7 pad 1: /Daughterboard/GPIO31 -> /Daughterboard/BTN_V4
- SW7 pad 2: Net-(D4-A) -> Net-(D16-A)
- SW8 pad 1: /Daughterboard/GPIO28 -> /Daughterboard/BTN_V1
- SW8 pad 2: Net-(D5-A) -> Net-(D1-A)
- SW9 pad 1: /Daughterboard/GPIO29 -> /Daughterboard/BTN_V2
- SW9 pad 2: Net-(D6-A) -> Net-(D2-A)
- U6 pad 2: unconnected-(U6-CAPP-Pad2) -> Net-(U6-CAPP)
- U6 pad 4: unconnected-(U6-CAPM-Pad4) -> Net-(U6-CAPM)
- U6 pad 6: /Daughterboard/AMP_L -> Net-(U6-OUTL)
- U6 pad 7: /Daughterboard/AMP_R -> Net-(U6-OUTR)
- U6 pad 8: +3V3 -> AVDD
- U6 pad 9: GND -> AGND
- U7 pad 13: +3V3 -> AVDD
- U7 pad 15: GND -> AGND
- U7 pad 2: GND -> AGND
- U7 pad 4: +3V3 -> AVDD
- U8 pad 13: +3V3 -> AVDD
- U8 pad 15: GND -> AGND
- U8 pad 2: GND -> AGND
- U8 pad 4: +3V3 -> AVDD
Routing:
- net (no net): track 1262.3 -> 0.00 mm
- net /Daughterboard/BTN_V2: track 0.00 -> 260.7 mm, vias 0 -> 2
- net /Daughterboard/BTN_V4: track 0.00 -> 250.5 mm, vias 0 -> 2
- net /Daughterboard/BTN_H3: track 0.00 -> 241.5 mm, vias 0 -> 1
- net /Daughterboard/BTN_V1: track 0.00 -> 233.9 mm, vias 0 -> 2
- net /Daughterboard/BTN_V3: track 0.00 -> 230.8 mm, vias 0 -> 2
- net /Daughterboard/BTN_H4: track 0.00 -> 203.4 mm, vias 0 -> 1
- net GND: track 154.8 -> 31.2 mm
- net /Daughterboard/BTN_H1: track 0.00 -> 60.8 mm, vias 0 -> 2
- net /Daughterboard/BTN_H2: track 0.00 -> 48.4 mm, vias 0 -> 2
- net /Daughterboard/GPIO39: track 53.2 -> 10.1 mm, vias 2 -> 0
- net /Daughterboard/GPIO32: track 18.1 -> 44.5 mm
- net /Daughterboard/GPIO35: track 19.1 -> 45.2 mm
- net Net-(D8-A): track 6.50 -> 30.0 mm, vias 0 -> 1
- net /Daughterboard/AMP_L: track 23.2 -> 0.00 mm, vias 2 -> 0
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Other:
- outline, holes or cut-outs redrawn
- board text added: "HSTX*8 3V3 GND"
- board text removed: "HSTX 3V3 GND"

Commit message: v2.0.0 WIP
Parts:
- removed R26: 0, Resistor_SMD:R_0402_1005Metric_Pad0.72x0.64mm_HandSolder
- added C42: 1u, Capacitor_SMD:C_0402_1005Metric_Pad0.74x0.62mm_HandSolder, B.Cu at (146.1, 41.3)
- added C43: 10u, Capacitor_SMD:C_0402_1005Metric_Pad0.74x0.62mm_HandSolder, B.Cu at (140.3, 47.0)
- added C44: 47n, Capacitor_SMD:C_0402_1005Metric_Pad0.74x0.62mm_HandSolder, B.Cu at (142.9, 41.9)
- added C45: 10u, Capacitor_SMD:C_0402_1005Metric_Pad0.74x0.62mm_HandSolder, B.Cu at (141.0, 44.5)
- added C46: 4.7u, Capacitor_SMD:C_0402_1005Metric_Pad0.74x0.62mm_HandSolder, B.Cu at (144.8, 41.3)
- added J7: Conn_01x04_MountingPin, Connector_JST:JST_SH_SM04B-SRSS-TB_1x04-1MP_P1.00mm_Horizontal, B.Cu at (83.2, 28.6)
- added LED6: GREEN, LED_SMD:LED_0805_2012Metric_Pad1.15x1.40mm_HandSolder, F.Cu at (154.9, 40.0)
- added R27: 10k, Resistor_SMD:R_0402_1005Metric_Pad0.72x0.64mm_HandSolder, B.Cu at (144.8, 48.9)
- added R28: 10k, Resistor_SMD:R_0402_1005Metric_Pad0.72x0.64mm_HandSolder, B.Cu at (78.1, 74.9)
- added R29: 10k, Resistor_SMD:R_0402_1005Metric_Pad0.72x0.64mm_HandSolder, B.Cu at (76.8, 74.9)
- added R30: 10k, Resistor_SMD:R_0402_1005Metric_Pad0.72x0.64mm_HandSolder, B.Cu at (75.6, 29.2)
- added R31: 10k, Resistor_SMD:R_0402_1005Metric_Pad0.72x0.64mm_HandSolder, B.Cu at (75.6, 27.9)
- added R32: 10k, Resistor_SMD:R_0402_1005Metric_Pad0.72x0.64mm_HandSolder, B.Cu at (74.3, 82.5)
- added R33: 10k, Resistor_SMD:R_0402_1005Metric_Pad0.72x0.64mm_HandSolder, B.Cu at (146.1, 48.9)
- added R34: 1k, Resistor_SMD:R_0402_1005Metric_Pad0.72x0.64mm_HandSolder, B.Cu at (154.9, 44.5)
- added TEMP1: temperture, Connector_Molex:Molex_PicoBlade_53261-0271_1x02-1MP_P1.25mm_Horizontal, B.Cu at (148.6, 34.3)
- added TP32: TP, TestPoint:TestPoint_Pad_D1.0mm, B.Cu at (123.7, 99.3)
- added TP33: TP, TestPoint:TestPoint_Pad_D1.0mm, B.Cu at (121.9, 98.3)
- added TP34: TP, TestPoint:TestPoint_Pad_D1.0mm, B.Cu at (141.9, 48.6)
- added U10: BQ25619, Package_DFN_QFN:Texas_RTW_WQFN-24-1EP_4x4mm_P0.5mm_EP2.7x2.7mm, B.Cu at (144.1, 45.1)
- added U9: MPU-6050, Sensor_Motion:InvenSense_QFN-24_4x4mm_P0.5mm, B.Cu at (76.2, 78.9)
- R12, R13, R14, R15: value 1k -> 10k
- R20, R21, R22, R23: footprint Resistor_SMD:R_0805_2012Metric_Pad1.20x1.40mm_HandSolder -> Resistor_SMD:R_0402_1005Metric_Pad0.72x0.64mm_HandSolder
- moved D14 110.6 mm to (50.2, 39.4)
- moved D15 33.0 mm to (54.6, 96.5)
- moved D16 24.2 mm to (52.1, 39.4), turned to 90 degrees
- moved D8 14.0 mm to (161.3, 96.5)
- moved SW16 7.91 mm to (52.0, 28.9), turned to 0 degrees
- moved BAT1 3.18 mm to (137.8, 34.3)
- moved D13 3.17 mm to (54.0, 39.4)
- moved TP15 2.69 mm to (121.9, 100.3)
- moved R24 0.13 mm to (129.5, 87.6)
- moved R25 0.13 mm to (129.5, 86.4)
Connections:
- net /Daughterboard/MAIN_GPIO12 renamed /Daughterboard/GPIO5
- net /Daughterboard/MAIN_GPIO13 renamed /Daughterboard/GPIO4
- D1 pad 1: /Daughterboard/BTN_H1 -> /Daughterboard/GPIO33
- D10 pad 1: /Daughterboard/BTN_H3 -> /Daughterboard/GPIO35
- D11 pad 1: /Daughterboard/BTN_H3 -> /Daughterboard/GPIO35
- D12 pad 1: /Daughterboard/BTN_H3 -> /Daughterboard/GPIO35
- D13 pad 1: /Daughterboard/BTN_H4 -> /Daughterboard/GPIO32
- D14 pad 1: /Daughterboard/BTN_H4 -> /Daughterboard/GPIO32
- D15 pad 1: /Daughterboard/BTN_H4 -> /Daughterboard/GPIO32
- D16 pad 1: /Daughterboard/BTN_H4 -> /Daughterboard/GPIO32
- D2 pad 1: /Daughterboard/BTN_H1 -> /Daughterboard/GPIO33
- D3 pad 1: /Daughterboard/BTN_H1 -> /Daughterboard/GPIO33
- D4 pad 1: /Daughterboard/BTN_H1 -> /Daughterboard/GPIO33
- D5 pad 1: /Daughterboard/BTN_H2 -> /Daughterboard/GPIO30
- D6 pad 1: /Daughterboard/BTN_H2 -> /Daughterboard/GPIO30
- D7 pad 1: /Daughterboard/BTN_H2 -> /Daughterboard/GPIO30
- D8 pad 1: /Daughterboard/BTN_H2 -> /Daughterboard/GPIO30
- D9 pad 1: /Daughterboard/BTN_H3 -> /Daughterboard/GPIO35
- SW10 pad 1: /Daughterboard/BTN_V3 -> /Daughterboard/GPIO31
- SW11 pad 1: /Daughterboard/BTN_V4 -> /Daughterboard/GPIO28
- SW12 pad 1: /Daughterboard/BTN_V1 -> /Daughterboard/GPIO29
- SW13 pad 1: /Daughterboard/BTN_V2 -> /Daughterboard/GPIO34
- SW14 pad 1: /Daughterboard/BTN_V3 -> /Daughterboard/GPIO31
- SW15 pad 1: /Daughterboard/BTN_V4 -> /Daughterboard/GPIO28
- SW16 pad 1: /Daughterboard/BTN_V1 -> /Daughterboard/GPIO29
- SW17 pad 1: /Daughterboard/BTN_V3 -> /Daughterboard/GPIO31
- SW18 pad 1: /Daughterboard/BTN_V3 -> /Daughterboard/GPIO31
- SW19 pad 1: /Daughterboard/BTN_V4 -> /Daughterboard/GPIO28
- SW4 pad 1: /Daughterboard/BTN_V2 -> /Daughterboard/GPIO34
- SW5 pad 1: /Daughterboard/BTN_V1 -> /Daughterboard/GPIO29
- SW6 pad 1: /Daughterboard/BTN_V2 -> /Daughterboard/GPIO34
- SW7 pad 1: /Daughterboard/BTN_V4 -> /Daughterboard/GPIO28
- SW8 pad 1: /Daughterboard/BTN_V1 -> /Daughterboard/GPIO29
- SW9 pad 1: /Daughterboard/BTN_V2 -> /Daughterboard/GPIO34
Routing:
- net /Daughterboard/GPIO28: track 54.1 -> 378.7 mm, vias 0 -> 4
- net /Daughterboard/GPIO34: track 45.1 -> 340.5 mm, vias 0 -> 4
- net /Daughterboard/GPIO31: track 45.1 -> 329.1 mm, vias 0 -> 4
- net /Daughterboard/BTN_V2: track 260.7 -> 0.00 mm, vias 2 -> 0
- net /Daughterboard/GPIO35: track 45.2 -> 298.6 mm, vias 0 -> 2
- net /Daughterboard/GPIO29: track 53.2 -> 305.3 mm, vias 0 -> 4
- net /Daughterboard/BTN_V4: track 250.5 -> 0.00 mm, vias 2 -> 0
- net /Daughterboard/BTN_H3: track 241.5 -> 0.00 mm, vias 1 -> 0
- net /Daughterboard/BTN_V1: track 233.9 -> 0.00 mm, vias 2 -> 0
- net /Daughterboard/BTN_V3: track 230.8 -> 0.00 mm, vias 2 -> 0
- net /Daughterboard/GPIO32: track 44.5 -> 272.3 mm, vias 0 -> 3
- net /Daughterboard/BTN_H4: track 203.4 -> 0.00 mm, vias 1 -> 0
- net /Daughterboard/GPIO30: track 45.1 -> 120.3 mm, vias 0 -> 3
- net /Daughterboard/GPIO21: track 12.7 -> 86.4 mm, vias 0 -> 2
- net /Daughterboard/GPIO33: track 45.0 -> 117.9 mm, vias 0 -> 2
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- added copper zone on B.Cu, net BAT_SW
- added copper zone on B.Cu, net VBAT
- added copper zone on B.Cu, net VSYS
- added copper zone on B.Cu, net VUSB
Other:
- outline, holes or cut-outs redrawn
- board text added: "CHARGING"
- board text added: "GPIO45"
- board text added: "GPIO46"
- board text added: "Z"
- board text added: "microSD/Qwiic"
- board text removed: "Battery"
- board text removed: "microSD"

Commit message: routing complete
Parts:
- added C47: 100n, Capacitor_SMD:C_0402_1005Metric_Pad0.74x0.62mm_HandSolder, B.Cu at (74.9, 80.6)
- added C48: 2.2n, Capacitor_SMD:C_0402_1005Metric_Pad0.74x0.62mm_HandSolder, B.Cu at (73.7, 73.7)
- added C49: 1u, Capacitor_SMD:C_0402_1005Metric_Pad0.74x0.62mm_HandSolder, B.Cu at (76.2, 80.6)
- added C50: 1u, Capacitor_SMD:C_0402_1005Metric_Pad0.74x0.62mm_HandSolder, B.Cu at (71.8, 75.6)
- added C51: 100n, Capacitor_SMD:C_0402_1005Metric_Pad0.74x0.62mm_HandSolder, B.Cu at (139.1, 90.2)
- added C52: 10u, Capacitor_SMD:C_0402_1005Metric_Pad0.74x0.62mm_HandSolder, B.Cu at (137.2, 92.1)
- added C54: 10u, Capacitor_SMD:C_0402_1005Metric_Pad0.74x0.62mm_HandSolder, B.Cu at (130.2, 85.1)
- added C55: 10u, Capacitor_SMD:C_0402_1005Metric_Pad0.74x0.62mm_HandSolder, B.Cu at (130.2, 90.2)
- added FB1: FerriteBead_Small, Inductor_SMD:L_0805_2012Metric_Pad1.15x1.40mm_HandSolder, B.Cu at (134.0, 92.1)
- added FB2: FerriteBead_Small, Inductor_SMD:L_0805_2012Metric_Pad1.15x1.40mm_HandSolder, B.Cu at (58.4, 97.8)
- added FB3: FerriteBead_Small, Inductor_SMD:L_0805_2012Metric_Pad1.15x1.40mm_HandSolder, B.Cu at (141.0, 97.9)
- added JP6: Jumper_2_Small_Bridged, Jumper:SolderJumper-2_P1.3mm_Bridged_Pad1.0x1.5mm, F.Cu at (128.3, 86.4)
- added JP7: Jumper_2_Small_Bridged, Jumper:SolderJumper-2_P1.3mm_Bridged_Pad1.0x1.5mm, F.Cu at (66.7, 100.8)
- added JP8: Jumper_2_Small_Bridged, Jumper:SolderJumper-2_P1.3mm_Bridged_Pad1.0x1.5mm, F.Cu at (149.2, 101.0)
- added L2: 1u, Inductor_SMD:L_6.3x6.3_H3, B.Cu at (139.7, 48.9)
- added Q1: SS8050, Package_TO_SOT_SMD:SOT-23, B.Cu at (105.4, 74.3)
- added R26: 10k, Resistor_SMD:R_0402_1005Metric_Pad0.72x0.64mm_HandSolder, B.Cu at (73.7, 80.6)
- added R35: 100, Resistor_SMD:R_0402_1005Metric_Pad0.72x0.64mm_HandSolder, B.Cu at (103.5, 72.4)
- added R36: 10k, Resistor_SMD:R_0402_1005Metric_Pad0.72x0.64mm_HandSolder, B.Cu at (106.0, 71.8)
- added R37: 1k, Resistor_SMD:R_0402_1005Metric_Pad0.72x0.64mm_HandSolder, B.Cu at (106.0, 70.5)
- added TP35: TP, TestPoint:TestPoint_Pad_D1.0mm, B.Cu at (83.7, 35.4)
- added TP36: TP, TestPoint:TestPoint_Pad_D1.0mm, B.Cu at (84.7, 33.7)
- added TP37: TP, TestPoint:TestPoint_Pad_D1.0mm, B.Cu at (141.4, 36.8)
- added TP38: TP, TestPoint:TestPoint_Pad_D1.0mm, B.Cu at (137.5, 40.5)
- added TP39: TP, TestPoint:TestPoint_Pad_D1.0mm, B.Cu at (138.0, 53.3)
- added TP40: TP, TestPoint:TestPoint_Pad_D1.0mm, B.Cu at (143.4, 36.8)
- C27, C28, C31, C32: value 470u -> 1u
- C39, C40: value 2.2u -> 2.2n
- NTC1: renamed from TEMP1; value temperture -> Temperture
- moved BAT1 23.6 mm to (140.3, 57.8)
- moved NTC1 23.6 mm to (151.1, 57.8)
- moved TP27 12.0 mm to (185.7, 79.5), turned to -90 degrees
- moved TP25 12.0 mm to (185.7, 81.5), turned to -90 degrees
- moved C31 10.5 mm to (154.3, 99.1), turned to 0 degrees
- moved C32 10.2 mm to (144.1, 99.1), turned to 180 degrees
- moved R33 9.55 mm to (146.7, 39.4), turned to 0 degrees
- moved TP26 9.20 mm to (185.7, 77.5), turned to -90 degrees
- moved R27 8.47 mm to (146.7, 40.6), turned to 0 degrees
- moved C40 8.26 mm to (124.5, 93.3), turned to 0 degrees
- moved R28 8.13 mm to (78.1, 83.1), turned to 180 degrees
- moved R29 7.10 mm to (78.1, 81.9), turned to 180 degrees
- moved C42 6.84 mm to (139.7, 38.7)
- moved R25 6.75 mm to (125.1, 91.4), turned to -90 degrees
- moved C46 6.48 mm to (138.4, 42.5), turned to -90 degrees
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Connections:
- net /Daughterboard/GPIO4 renamed /Daughterboard/MAIN_GPIO13
- net /Daughterboard/GPIO5 renamed /Daughterboard/MAIN_GPIO12
- net Net-(U10-~{CE}) renamed /Daughterboard/~{BAT_CE}
- AUDIO1 pad S: AGND -> GND
- C27 pad 1: +3V3 -> AVDD
- C27 pad 2: GND -> AGND
- C28 pad 1: +3V3 -> AVDD
- C28 pad 2: GND -> AGND
- C31 pad 1: +3V3 -> AVDD
- C31 pad 2: GND -> AGND
- C32 pad 1: +3V3 -> AVDD
- C32 pad 2: GND -> AGND
- C38 pad 1: unconnected-(C38-Pad1) -> Net-(U6-VNEG)
- C38 pad 2: unconnected-(C38-Pad2) -> AGND
- C39 pad 1: /Daughterboard/DAC_L -> AGND
- C39 pad 2: AGND -> /Daughterboard/DAC_L
- C40 pad 1: /Daughterboard/DAC_R -> AGND
- C40 pad 2: AGND -> /Daughterboard/DAC_R
- U10 pad 2: unconnected-(U10-PSEL-Pad2) -> Net-(U10-PSEL)
- U10 pad 23: unconnected-(U10-PMID-Pad23) -> Net-(U10-PMID)
- U10 pad 3: unconnected-(U10-PMID_GOOD-Pad3) -> Net-(U10-PMID_GOOD)
- U6 pad 1: +3V3 -> AVDD
- U6 pad 18: unconnected-(U6-LDOO-Pad18) -> Net-(U6-LDOO)
- U6 pad 3: GND -> AGND
- U6 pad 5: unconnected-(U6-VNEG-Pad5) -> Net-(U6-VNEG)
- U9 pad 1: unconnected-(U9-CLKIN-Pad1) -> GND
- U9 pad 10: unconnected-(U9-REGOUT-Pad10) -> Net-(U9-REGOUT)
- U9 pad 11: unconnected-(U9-FSYNC-Pad11) -> Net-(U9-FSYNC)
- U9 pad 20: unconnected-(U9-CPOUT-Pad20) -> Net-(U9-CPOUT)
Routing:
- net /Daughterboard/GPIO25: track 6.86 -> 98.6 mm, vias 0 -> 4
- net /Daughterboard/GPIO22: track 50.8 -> 140.1 mm, vias 1 -> 6
- net /Daughterboard/GPIO23: track 52.7 -> 141.7 mm, vias 1 -> 6
- net AGND: track 18.0 -> 65.8 mm, vias 6 -> 13
- net +3V3: track 504.3 -> 551.7 mm, vias 23 -> 33
- net /Daughterboard/GPIO36: track 10.1 -> 46.3 mm, vias 0 -> 2
- net /Daughterboard/GPIO38: track 10.1 -> 43.9 mm, vias 0 -> 2
- net /Daughterboard/GPIO37: track 10.3 -> 43.9 mm, vias 0 -> 2
- net /Daughterboard/GPIO39: track 10.1 -> 43.5 mm, vias 0 -> 2
- net /Daughterboard/GPIO9: track 71.0 -> 104.1 mm
- net AVDD: track 0.00 -> 29.0 mm, vias 0 -> 4
- net /Daughterboard/DAC_L: track 0.22 -> 28.9 mm, vias 1 -> 2
- net /Daughterboard/DAC_R: track 0.00 -> 17.8 mm, vias 1 -> 2
- net VUSB: track 150.0 -> 133.4 mm
- net /Daughterboard/GPIO24: track 27.3 -> 43.3 mm
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- added copper zone on B.Cu, net AVDD
- added copper zone on F.Cu, net VBAT
Other:
- board text added: "LS"
- board text added: "LX"
- board text added: "LY"
- board text added: "PG"
- board text added: "PICO CONSOLE V2"
- board text added: "PMID"
- board text added: "PSEL"
- board text added: "RS"
- board text added: "RX"
- board text added: "RY"
- board text added: "SCL"
- board text added: "SDA"
- board text added: "VSYS"
- board text added: "~{QON}"
- board text removed: "V2"
