File: pico_concole_v2_daughter_board.kicad_sch (KiCad schematic)
At the start: 0 parts

Commit message: Place components temporarily
Changed lines of the file:
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@@
 	(text "VUSB : 5.0V (typical)\nVIN  : 5.2 - 3.0V\nVBAT : 4.2 - 3.0V\n3V3  : 3.3V (typical)"
 		(exclude_from_sim no)
-		(at 127.254 29.972 0)
+		(at 114.554 29.972 0)
 		(effects
 			(font

Commit message: v2.0.0 WIP
Other:
- sheet Daughterboard ports: added ~{SB_RUN}; removed none
- sheet Southbridge ports: added ~{SB_RUN}; removed none
Changed lines of the file:
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@@
+		)
+	)
+	(bus
+		(pts
+			(xy 50.8 68.58) (xy 63.5 68.58)
+		)
+		(stroke
+			(width 0)
+			(type default)
 		)
 	)
 	(wire
 		(pts
+			(xy 50.8 66.04) (xy 63.5 66.04)
+		)
+		(stroke
+			(width 0)
+			(type default)
+		)
+	)
+	(wire
+		(pts
 			(xy 50.8 27.94) (xy 63.5 27.94)
-		)
-		(stroke
-			(width 0)
-			(type default)
-		)
-	)
-	(bus
-		(pts
-			(xy 50.8 66.04) (xy 63.5 66.04)
 		)
 		(stroke
@@
 		)
 		(pin "GPIO[02..47]" bidirectional
-			(at 63.5 66.04 180)
+			(at 63.5 68.58 180)
 			(effects
 				(font
@@
 		(pin "~{MAIN_RUN}" output
 			(at 63.5 27.94 180)
+			(effects
+				(font
+					(size 1.27 1.27)
+				)
+				(justify left)
+			)
+		)
+		(pin "~{SB_RUN}" output
+			(at 63.5 66.04 180)
 			(effects
 				(font
@@
 		)
 		(pin "GPIO[02..47]" bidirectional
+			(at 50.8 68.58 0)
+			(effects
+				(font
+					(size 1.27 1.27)
+				)
+				(justify right)
+			)
+		)
+		(pin "~{SB_RUN}" input
 			(at 50.8 66.04 0)
 			(effects

Commit message: v2.0.0 WIP
Other:
- note added: "VUSB : 5.0V (typical) VIN : 5.5 - 3.0V VBAT : 4.2 - 3.0V 3V3 : 3.3V (typical)"
- note removed: "VUSB : 5.0V (typical) VIN : 5.2 - 3.0V VBAT : 4.2 - 3.0V 3V3 : 3.3V (typical)"
Changed lines of the file:
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@@
 	(generator_version "9.0")
 	(paper "A4")
-	(text "VUSB : 5.0V (typical)\nVIN  : 5.2 - 3.0V\nVBAT : 4.2 - 3.0V\n3V3  : 3.3V (typical)"
+	(text "VUSB : 5.0V (typical)\nVIN  : 5.5 - 3.0V\nVBAT : 4.2 - 3.0V\n3V3  : 3.3V (typical)"
 		(exclude_from_sim no)
 		(at 114.554 29.972 0)
