File: Southbridge.kicad_sch (KiCad schematic)
At the start: 6 parts, among them J1 USB_C_Receptacle_USB2.0_16P, J2 SM03B-SRSS-TB, J3 SM03B-SRSS-TB, U3 RP2350_80QFN

Commit message: Place components temporarily
Changed lines of the file:
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@@
+	)
+	(symbol
+		(lib_id "power:+3.3V")
+		(at 203.2 64.77 0)
+		(unit 1)
+		(exclude_from_sim no)
+		(in_bom yes)
+		(on_board yes)
+		(dnp no)
+		(property "Reference" "#PWR047"
+			(at 203.2 68.58 0)
+			(effects
+				(font
+					(size 1.27 1.27)
+				)
+				(hide yes)
+			)
+		)
+		(property "Value" "+3V3"
+			(at 202.946 60.96 0)
+			(effects
+				(font
+					(size 1.27 1.27)
+				)
+			)
+		)
+		(property "Footprint" ""
+			(at 203.2 64.77 0)
+			(effects
+				(font
+					(size 1.27 1.27)
+				)
+				(hide yes)
+			)
+		)
+		(property "Datasheet" ""
+			(at 203.2 64.77 0)
+			(effects
+				(font
+					(size 1.27 1.27)
+				)
+				(hide yes)
+			)
+		)
+		(property "Description" "Power symbol creates a global label with name \"+3.3V\""
+			(at 203.2 64.77 0)
+			(effects
+				(font
+					(size 1.27 1.27)
+				)
+				(hide yes)
+			)
+		)
+		(pin "1"
+		)
+		(instances
+			(project "pico_concole_v2_daughter_board"
+				(path "/aa71e631-a14f-409f-b19b-1d980ff58830/4f2d6bec-4cdf-405c-a073-de4a6062ff14"
+					(reference "#PWR047")
+					(unit 1)
+				)
+			)
+		)
 	)
 	(symbol
@@
 					(unit 1)
 				)
+			)
+		)
+	)
+	(symbol
+		(lib_id "power:+3.3V")
+		(at 209.55 64.77 0)
+		(unit 1)
+		(exclude_from_sim no)
+		(in_bom yes)
+		(on_board yes)
+		(dnp no)
+		(property "Reference" "#PWR048"
+			(at 209.55 68.58 0)
+			(effects
+				(font
+					(size 1.27 1.27)
+				)
+				(hide yes)
+			)
+		)
+		(property "Value" "+1V1"
+			(at 209.296 60.96 0)
+			(effects
+				(font
+					(size 1.27 1.27)
+				)
+			)
+		)
+		(property "Footprint" ""
+			(at 209.55 64.77 0)
+			(effects
+				(font
+					(size 1.27 1.27)
+				)
+				(hide yes)
+			)
+		)
+		(property "Datasheet" ""
+			(at 209.55 64.77 0)
+			(effects
+				(font
+					(size 1.27 1.27)
+				)
+				(hide yes)
+			)
+		)
+		(property "Description" "Power symbol creates a global label with name \"+3.3V\""
+			(at 209.55 64.77 0)
+			(effects
+				(font
+					(size 1.27 1.27)
+				)
+				(hide yes)
+			)
+		)
+		(pin "1"
+		)
+		(instances
+			(project "pico_concole_v2_daughter_board"
+				(path "/aa71e631-a14f-409f-b19b-1d980ff58830/4f2d6bec-4cdf-405c-a073-de4a6062ff14"
+					(reference "#PWR048")
+					(unit 1)
+				)

Commit message: v2.0.0 WIP
Parts:
- renumbered U3 to U1
Connections:
- net GPIO40_ADC0 renamed GPIO40
- net GPIO41_ADC1 renamed GPIO41
- net GPIO42_ADC2 renamed GPIO42
- net GPIO43_ADC3 renamed GPIO43
- net GPIO44_ADC4 renamed GPIO44
- net GPIO45_ADC5 renamed GPIO45
- net GPIO46_ADC6 renamed GPIO46
- net GPIO47_ADC7 renamed GPIO47

Commit message: v2.0.0 WIP
Parts:
- added C1, C10, C11, C12, C16, C2, C3, C4, C5, C6, C7, C8, C9: 100n, Capacitor_SMD:C_0402_1005Metric_Pad0.74x0.62mm_HandSolder, symbol Device:C
- added C13, C14, C15: 4.7u, Capacitor_SMD:C_0603_1608Metric_Pad1.08x0.95mm_HandSolder, symbol Device:C
- added C17, C18: 15p, Capacitor_SMD:C_0402_1005Metric_Pad0.74x0.62mm_HandSolder, symbol Device:C
- added L1: AOTA-B201610S3R3-101-T, inductor:L_pol_2016, symbol Device:L
- added R3: 33, Resistor_SMD:R_0603_1608Metric_Pad0.98x0.95mm_HandSolder, symbol Device:R
- added R4, R5: 27, Resistor_SMD:R_0402_1005Metric_Pad0.72x0.64mm_HandSolder, symbol Device:R
- added R6, R7, R8: 1k, Resistor_SMD:R_0402_1005Metric_Pad0.72x0.64mm_HandSolder, symbol Device:R
- added SW1, SW2: SW_Push, Button_Switch_SMD:SW_Push_1P1T_NO_Vertical_Wuerth_434133025816, symbol Switch:SW_Push
- added U2: W25Q16JVSS, Package_SO:SOIC-8_5.3x5.3mm_P1.27mm, symbol Memory_Flash:W25Q16JVSS
- added Y1: ABM8-272-T3, Crystal:Crystal_SMD_3225-4Pin_3.2x2.5mm, symbol Device:Crystal_GND24
- renumbered J2 to J1, J3 to J2, J1 to J3
Connections:
- net +1V1: now also U1.10 (DVDD), U1.32 (DVDD), U1.51 (DVDD), U1.65 (VREG_FB), C1.1, C15.1, C2.1, C3.1, L1.1
- net +3V3: now also U1.15 (IOVDD), U1.24 (IOVDD), U1.29 (IOVDD), U1.41 (IOVDD), U1.5 (IOVDD), U1.50 (IOVDD), U1.59 (ADC_AVDD), U1.60 (IOVDD), U1.64 (VREG_VIN), U1.68 (USB_OTP_VDD), U1.69 (QSPI_IOVDD), U1.76 (IOVDD), C10.1, C11.1, C12.1, C14.1, C16.1, C4.1, C5.1, C6.1, C7.1, C8.1, C9.1, R3.1, U2.8 (VCC)
- net GND: now also U1.62 (VREG_PGND), U1.81 (GND), C1.2, C10.2, C11.2, C12.2, C13.2, C14.2, C15.2, C16.2, C17.2, C18.2, C2.2, C3.2, C4.2, C5.2, C6.2, C7.2, C8.2, C9.2, R7.1, SW1.1, U2.4 (GND), Y1.2, Y1.4
- net QSPI_SCLK: now also U2.6 (CLK)
- net QSPI_SD0: now also U2.5 (DI/IO_{0})
- net QSPI_SD1: now also U2.2 (DO/IO_{1})
- net QSPI_SD2: now also U2.3 (~{WP}/IO_{2})
- net QSPI_SD3: now also U2.7 (~{HOLD}/~{RESET}/IO_{3})
- net QSPI_SS: now also R6.2, U2.1 (~{CS})
- net USB_D+: now also R4.2
- net USB_D-: now also R5.2
- net XIN: now also C17.1, Y1.1
- net XOUT: now also R8.1
- net VREG_AVDD: now reaches U1.61 (VREG_AVDD)
- net VREG_AVDD: now also C13.1, R3.2
- net VREG_LX: now reaches U1.63 (VREG_LX)
- net VREG_LX: now also L1.2
- net RP2350_D-: now reaches U1.66 (USB_DM)
- net RP2350_D-: now also R5.1
- net RP2350_D+: now reaches U1.67 (USB_DP)
- net RP2350_D+: now also R4.1
- net RUN renamed ~{SB_RUN}
- net ~{SB_RUN}: now also SW2.2
- new net: R7.2, SW2.1
- new net: C18.1, R8.2, Y1.3
- new net ~{USB_BOOT}: R6.1, SW1.2
Other:
- note added: "FLASH"
- moved on the sheet: U1

Commit message: v2.0.0 WIP
Parts:
- L1: footprint inductor:L_pol_2016 -> Library:L_pol_2016
- R3: footprint Resistor_SMD:R_0603_1608Metric_Pad0.98x0.95mm_HandSolder -> Capacitor_SMD:C_0402_1005Metric_Pad0.74x0.62mm_HandSolder
- U1: footprint Library:QFN-80-1EP_10x10mm_P0.4mm_EP3.4x3.4mm_ThermalVias -> Package_DFN_QFN:QFN-80-1EP_10x10mm_P0.4mm_EP3.4x3.4mm
Changed lines of the file:
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@@
 			)
 		)
-		(property "Footprint" "Library:QFN-80-1EP_10x10mm_P0.4mm_EP3.4x3.4mm_ThermalVias"
+		(property "Footprint" "Package_DFN_QFN:QFN-80-1EP_10x10mm_P0.4mm_EP3.4x3.4mm"
 			(at 101.6 180.34 0)
 			(effects
@@
 			)
 		)
-		(property "Footprint" "Resistor_SMD:R_0603_1608Metric_Pad0.98x0.95mm_HandSolder"
+		(property "Footprint" "Capacitor_SMD:C_0402_1005Metric_Pad0.74x0.62mm_HandSolder"
 			(at 64.77 127.508 90)
 			(effects
@@
 			)
 		)
-		(property "Footprint" "inductor:L_pol_2016"
+		(property "Footprint" "Library:L_pol_2016"
 			(at 57.15 143.51 0)
 			(effects

Commit message: V2.0.0 WIP
Parts:
- added U1: USBLC6-2SC6, Package_TO_SOT_SMD:SOT-23-6, symbol Power_Protection:USBLC6-2SC6
- renumbered U1 to U2, U2 to U3
Connections:
- net GND: now also U1.2 (GND)
- net USB_D+: now also U1.3 (I/O2), U1.4 (I/O2)
- net USB_D-: now also U1.1 (I/O1), U1.6 (I/O1)
- net VBUS renamed VUSB
- net VUSB: now also U1.5 (VBUS)

Commit message: V2.0.0 WIP
Other:
- moved on the sheet: R4
Changed lines of the file:
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@@
 	(wire
 		(pts
-			(xy 160.02 134.62) (xy 160.02 137.16)
-		)
-		(stroke
-			(width 0)
-			(type default)
-		)
-	)
-	(wire
-		(pts
 			(xy 157.48 210.82) (xy 172.72 210.82)
 		)
@@
 	(wire
 		(pts
-			(xy 190.5 134.62) (xy 180.34 134.62)
+			(xy 190.5 137.16) (xy 180.34 137.16)
 		)
 		(stroke
@@
 	(wire
 		(pts
-			(xy 160.02 134.62) (xy 172.72 134.62)
-		)
-		(stroke
-			(width 0)
-			(type default)
-		)
-	)
-	(wire
-		(pts
 			(xy 157.48 139.7) (xy 172.72 139.7)
 		)
@@
 	(wire
 		(pts
-			(xy 160.02 137.16) (xy 157.48 137.16)
+			(xy 157.48 137.16) (xy 172.72 137.16)
 		)
 		(stroke
@@
 	)
 	(label "USB_D+"
-		(at 190.5 134.62 180)
+		(at 190.5 137.16 180)
 		(effects
 			(font
@@
 	)
 	(label "RP2350_D+"
-		(at 172.72 134.62 180)
+		(at 172.72 137.16 180)
 		(effects
 			(font
@@
 		(lib_id "Device:R")
 		(at 176.53 139.7 90)
+		(mirror x)
 		(unit 1)
 		(exclude_from_sim no)
@@
 		(dnp no)
 		(property "Reference" "R5"
-			(at 176.022 137.668 90)
+			(at 176.022 141.732 90)
 			(effects
 				(font
@@
 		)
 		(property "Value" "27"
-			(at 179.832 137.668 90)
+			(at 179.832 141.732 90)
 			(effects
 				(font
@@
 		)
 		(property "Footprint" "Resistor_SMD:R_0402_1005Metric_Pad0.72x0.64mm_HandSolder"
-			(at 176.53 141.478 90)
+			(at 176.53 137.922 90)
 			(effects
 				(font
@@
 	(symbol
 		(lib_id "Device:R")
-		(at 176.53 134.62 90)
+		(at 176.53 137.16 90)
 		(unit 1)
 		(exclude_from_sim no)
@@
 		(dnp no)
 		(property "Reference" "R4"
-			(at 176.022 132.588 90)
+			(at 176.022 135.128 90)
 			(effects
 				(font
@@
 		)
 		(property "Value" "27"
-			(at 179.832 132.588 90)
+			(at 179.832 135.128 90)
 			(effects
 				(font
@@
 		)
 		(property "Footprint" "Resistor_SMD:R_0402_1005Metric_Pad0.72x0.64mm_HandSolder"
-			(at 176.53 136.398 90)
+			(at 176.53 138.938 90)
 			(effects
 				(font
@@
 		)
 		(property "Datasheet" "~"
-			(at 176.53 134.62 0)
+			(at 176.53 137.16 0)
 			(effects
 				(font
@@
 		)
 		(property "Description" "Resistor"
-			(at 176.53 134.62 0)
+			(at 176.53 137.16 0)
 			(effects
 				(font

Commit message: Update BOM
Parts:
- R1, R2: now left out of the parts list
- R6, R7, R8: now in the parts list
- U2: LCSC PN (none) -> C42415655
Changed lines of the file:
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@@
 		(unit 1)
 		(exclude_from_sim no)
-		(in_bom yes)
+		(in_bom no)
 		(on_board yes)
 		(dnp no)
@@
 			)
 		)
+		(property "LCSC PN" "C42415655"
+			(at 120.65 180.34 0)
+			(effects
+				(font
+					(size 1.27 1.27)
+				)
+				(hide yes)
+			)
+		)
 		(pin "1"
 		)
@@
 		(unit 1)
 		(exclude_from_sim no)
-		(in_bom no)
+		(in_bom yes)
 		(on_board yes)
 		(dnp no)
@@
 		(unit 1)
 		(exclude_from_sim no)
-		(in_bom no)
+		(in_bom yes)
 		(on_board yes)
 		(dnp no)
@@
 		(unit 1)
 		(exclude_from_sim no)
-		(in_bom yes)
+		(in_bom no)
 		(on_board yes)
 		(dnp no)
@@
 		(unit 1)
 		(exclude_from_sim no)
-		(in_bom no)
+		(in_bom yes)
 		(on_board yes)
 		(dnp no)
